File: rescuetruck-main/MCU.kicad_sch (KiCad schematic)
At the start: 24 parts, among them IC1 W25Q16JVUXIQ, SW1 Reset, U3 RP2040, Y1 JGHC S3212000181080

Commit message: vootvan progress
Changed lines of the file:
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@@
     (effects (font (size 1.27 1.27)) (justify right bottom))
+  )
+  (global_label "SELECT1" (shape input) (at 142.24 124.46 180) (fields_autoplaced)
+    (effects (font (size 1.27 1.27)) (justify right))
+    (property "Intersheetrefs" "${INTERSHEET_REFS}" (at 132.0057 124.46 0)
+      (effects (font (size 1.27 1.27)) (justify right) hide)
+    )
+  )
+  (global_label "SELECT3" (shape input) (at 142.24 129.54 180) (fields_autoplaced)
+    (effects (font (size 1.27 1.27)) (justify right))
+    (property "Intersheetrefs" "${INTERSHEET_REFS}" (at 132.0057 129.54 0)
+      (effects (font (size 1.27 1.27)) (justify right) hide)
+    )
+  )
+  (global_label "SELECT0" (shape input) (at 142.24 121.92 180) (fields_autoplaced)
+    (effects (font (size 1.27 1.27)) (justify right))
+    (property "Intersheetrefs" "${INTERSHEET_REFS}" (at 132.0057 121.92 0)
+      (effects (font (size 1.27 1.27)) (justify right) hide)
+    )
+  )
+  (global_label "SELECT2" (shape input) (at 142.24 127 180) (fields_autoplaced)
+    (effects (font (size 1.27 1.27)) (justify right))
+    (property "Intersheetrefs" "${INTERSHEET_REFS}" (at 132.0057 127 0)
+      (effects (font (size 1.27 1.27)) (justify right) hide)
+    )
+  )
+  (global_label "AM0" (shape input) (at 142.24 111.76 180) (fields_autoplaced)
+    (effects (font (size 1.27 1.27)) (justify right))
+    (property "Intersheetrefs" "${INTERSHEET_REFS}" (at 136.2389 111.76 0)
+      (effects (font (size 1.27 1.27)) (justify right) hide)
+    )
+  )
+  (global_label "RGB MCU" (shape input) (at 141.986 104.394 180) (fields_autoplaced)
+    (effects (font (size 1.27 1.27)) (justify right))
+    (property "Intersheetrefs" "${INTERSHEET_REFS}" (at 131.1105 104.394 0)
+      (effects (font (size 1.27 1.27)) (justify right) hide)
+    )
   )
   (global_label "USB_D+" (shape input) (at 125.222 60.706 0) (fields_autoplaced)
@@
     )
   )
+  (global_label "AM2" (shape input) (at 142.24 116.84 180) (fields_autoplaced)
+    (effects (font (size 1.27 1.27)) (justify right))
+    (property "Intersheetrefs" "${INTERSHEET_REFS}" (at 136.2389 116.84 0)
+      (effects (font (size 1.27 1.27)) (justify right) hide)
+    )
+  )
   (global_label "USB_D-" (shape input) (at 125.222 68.326 0) (fields_autoplaced)
     (effects (font (size 1.27 1.27)) (justify left))
@@
     )
   )
+  (global_label "AM1" (shape input) (at 142.24 114.3 180) (fields_autoplaced)
+    (effects (font (size 1.27 1.27)) (justify right))
+    (property "Intersheetrefs" "${INTERSHEET_REFS}" (at 136.2389 114.3 0)
+      (effects (font (size 1.27 1.27)) (justify right) hide)
+    )
+  )

Commit message: continue progress
Connections:
- net ADC_X is gone; now on net AM0: U3.39 (GPIO27_ADC1)
- net GPIO17 is gone; now on net SELECT3: U3.28 (GPIO17)
- net GPIO20 is gone; now on net SELECT2: U3.31 (GPIO20)
- net GPIO23 is gone; now on net SELECT0: U3.35 (GPIO23)
- net GPIO25 is gone; now on net AM2: U3.37 (GPIO25)
- net GPIO29_ADC3 is gone; now on net AM1: U3.41 (GPIO29_ADC3)
- net GPIO6 is gone; now on net RGB MCU: U3.8 (GPIO6)
- net OLED_SDA is gone; now on net SELECT1: U3.29 (GPIO18)
- net ADC_Z renamed GPIO26_ADC0
- net OLED_SCL renamed GPIO19
- no-connect marks 29 -> 23
Other:
- note added: "Make sure C20 is close to pin 45 of RP2040"
- note added: "Make sure C21 is close to pin 44 of RP2040"
- note added: "Make sure R7 and R8 are close to RP2040"
- note removed: "Make sure C10 is close to pin 44 of RP2040"
- note removed: "Make sure C8 is close to pin 45 of RP2040"
- note removed: "Make sure R3 and R4 are close to RP2040"
Changed lines of the file:
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@@
   (no_connect (at 118.618 78.486))
   (no_connect (at 118.618 83.566))
-  (no_connect (at 118.618 152.146))
   (no_connect (at 118.618 96.266))
   (no_connect (at 118.618 81.026))
   (no_connect (at 118.618 86.106))
   (no_connect (at 118.618 108.966))
-  (no_connect (at 118.618 91.186))
-  (no_connect (at 118.618 136.906))
   (no_connect (at 118.618 116.586))
-  (no_connect (at 118.618 126.746))
+  (no_connect (at 118.618 124.206))
   (no_connect (at 118.618 129.286))
   (no_connect (at 118.618 103.886))
   (no_connect (at 118.618 93.726))
   (no_connect (at 25.908 129.286))
-  (no_connect (at 118.618 149.606))
   (no_connect (at 243.586 56.134))
   (no_connect (at 118.618 101.346))
-  (no_connect (at 118.618 119.126))
   (no_connect (at 118.618 111.506))
   (no_connect (at 118.618 131.826))
@@
   (no_connect (at 118.618 98.806))
   (no_connect (at 25.908 143.256))
-  (no_connect (at 118.618 139.446))
   (no_connect (at 118.618 75.946))
-  (no_connect (at 118.618 134.366))
+  (no_connect (at 118.5982 106.426))
   (no_connect (at 118.618 114.046))
   (no_connect (at 118.618 88.646))
@@
     (effects (font (size 2.54 2.54)) (justify left bottom))
   )
-  (text "Make sure C10 is close to pin 44 of RP2040" (at 104.648 48.006 0)
+  (text "Make sure C21 is close to pin 44 of RP2040" (at 104.648 48.006 0)
     (effects (font (size 1.27 1.27)) (justify left bottom))
   )
@@
     (effects (font (size 2.54 2.54)) (justify left bottom))
   )
-  (text "Make sure C8 is close to pin 45 of RP2040" (at -5.842 46.736 0)
-    (effects (font (size 1.27 1.27)) (justify left bottom))
-  )
-  (text "Make sure R3 and R4 are close to RP2040" (at 126.238 64.516 0)
-    (effects (font (size 1.27 1.27)) (justify left bottom))
+  (text "Make sure C20 is close to pin 45 of RP2040" (at -5.842 46.736 0)
+    (effects (font (size 1.27 1.27)) (justify left bottom))
+  )
+  (text "Make sure R7 and R8 are close to RP2040" (at 126.238 64.516 0)
+    (effects (font (size 1.27 1.27)) (justify left bottom))
+  )
+  (label "GPIO27_ADC1" (at 118.618 147.066 180) (fields_autoplaced)
+    (effects (font (size 1.27 1.27)) (justify right bottom))
   )
   (label "QSPI_SD0" (at 274.066 48.514 180) (fields_autoplaced)
@@
     (effects (font (size 1.27 1.27)) (justify left bottom))
   )
-  (label "OLED_SCL" (at 118.618 124.206 180) (fields_autoplaced)
+  (label "GPIO19" (at 118.618 124.206 180) (fields_autoplaced)
     (effects (font (size 1.27 1.27)) (justify right bottom))
   )
@@
     (effects (font (size 1.27 1.27)) (justify right bottom))
   )
-  (label "OLED_SDA" (at 118.618 121.666 180) (fields_autoplaced)
+  (label "GPIO26_ADC0" (at 118.618 144.526 180) (fields_autoplaced)
+    (effects (font (size 1.27 1.27)) (justify right bottom))
+  )
+  (label "GPIO18" (at 118.618 121.666 180) (fields_autoplaced)
     (effects (font (size 1.27 1.27)) (justify right bottom))
   )
@@
     (effects (font (size 1.27 1.27)) (justify right bottom))
   )
-  (global_label "SELECT1" (shape input) (at 142.24 124.46 180) (fields_autoplaced)
-    (effects (font (size 1.27 1.27)) (justify right))
-    (property "Intersheetrefs" "${INTERSHEET_REFS}" (at 132.0057 124.46 0)
-      (effects (font (size 1.27 1.27)) (justify right) hide)
-    )
-  )
-  (global_label "SELECT3" (shape input) (at 142.24 129.54 180) (fields_autoplaced)
-    (effects (font (size 1.27 1.27)) (justify right))
-    (property "Intersheetrefs" "${INTERSHEET_REFS}" (at 132.0057 129.54 0)
-      (effects (font (size 1.27 1.27)) (justify right) hide)
-    )
-  )
-  (global_label "SELECT0" (shape input) (at 142.24 121.92 180) (fields_autoplaced)
-    (effects (font (size 1.27 1.27)) (justify right))
-    (property "Intersheetrefs" "${INTERSHEET_REFS}" (at 132.0057 121.92 0)
-      (effects (font (size 1.27 1.27)) (justify right) hide)
-    )
-  )
-  (global_label "SELECT2" (shape input) (at 142.24 127 180) (fields_autoplaced)
-    (effects (font (size 1.27 1.27)) (justify right))
-    (property "Intersheetrefs" "${INTERSHEET_REFS}" (at 132.0057 127 0)
-      (effects (font (size 1.27 1.27)) (justify right) hide)
-    )
-  )
-  (global_label "AM0" (shape input) (at 142.24 111.76 180) (fields_autoplaced)
-    (effects (font (size 1.27 1.27)) (justify right))
-    (property "Intersheetrefs" "${INTERSHEET_REFS}" (at 136.2389 111.76 0)
-      (effects (font (size 1.27 1.27)) (justify right) hide)
-    )
-  )
-  (global_label "RGB MCU" (shape input) (at 141.986 104.394 180) (fields_autoplaced)
-    (effects (font (size 1.27 1.27)) (justify right))
-    (property "Intersheetrefs" "${INTERSHEET_REFS}" (at 131.1105 104.394 0)
-      (effects (font (size 1.27 1.27)) (justify right) hide)
+  (global_label "SELECT1" (shape input) (at 118.618 121.666 0) (fields_autoplaced)
+    (effects (font (size 1.27 1.27)) (justify left))
+    (property "Intersheetrefs" "${INTERSHEET_REFS}" (at 128.8523 121.666 0)
+      (effects (font (size 1.27 1.27)) (justify left) hide)
+    )
+  )
+  (global_label "SELECT3" (shape input) (at 118.618 119.126 0) (fields_autoplaced)
+    (effects (font (size 1.27 1.27)) (justify left))
+    (property "Intersheetrefs" "${INTERSHEET_REFS}" (at 128.8523 119.126 0)
+      (effects (font (size 1.27 1.27)) (justify left) hide)
+    )
+  )
+  (global_label "SELECT0" (shape input) (at 118.618 134.366 0) (fields_autoplaced)
+    (effects (font (size 1.27 1.27)) (justify left))
+    (property "Intersheetrefs" "${INTERSHEET_REFS}" (at 128.8523 134.366 0)
+      (effects (font (size 1.27 1.27)) (justify left) hide)
+    )
+  )
+  (global_label "SELECT2" (shape input) (at 118.618 126.746 0) (fields_autoplaced)
+    (effects (font (size 1.27 1.27)) (justify left))
+    (property "Intersheetrefs" "${INTERSHEET_REFS}" (at 128.8523 126.746 0)
+      (effects (font (size 1.27 1.27)) (justify left) hide)
+    )
+  )
+  (global_label "AM0" (shape input) (at 118.618 147.066 0) (fields_autoplaced)
+    (effects (font (size 1.27 1.27)) (justify left))
+    (property "Intersheetrefs" "${INTERSHEET_REFS}" (at 124.6191 147.066 0)
+      (effects (font (size 1.27 1.27)) (justify left) hide)
+    )
+  )
+  (global_label "RGB MCU" (shape input) (at 118.618 91.186 0) (fields_autoplaced)
+    (effects (font (size 1.27 1.27)) (justify left))
+    (property "Intersheetrefs" "${INTERSHEET_REFS}" (at 129.4935 91.186 0)
+      (effects (font (size 1.27 1.27)) (justify left) hide)
     )
   )
@@
     )
   )
-  (global_label "ADC_Z" (shape input) (at 118.618 144.526 0) (fields_autoplaced)
-    (effects (font (size 1.27 1.27)) (justify left))
-    (property "Intersheetrefs" "${INTERSHEET_REFS}" (at 127.3295 144.526 0)
-      (effects (font (size 1.27 1.27)) (justify left) hide)
-    )
-  )
-  (global_label "AM2" (shape input) (at 142.24 116.84 180) (fields_autoplaced)
-    (effects (font (size 1.27 1.27)) (justify right))
-    (property "Intersheetrefs" "${INTERSHEET_REFS}" (at 136.2389 116.84 0)
-      (effects (font (size 1.27 1.27)) (justify right) hide)
+  (global_label "AM2" (shape input) (at 118.618 139.446 0) (fields_autoplaced)
+    (effects (font (size 1.27 1.27)) (justify left))
+    (property "Intersheetrefs" "${INTERSHEET_REFS}" (at 124.6191 139.446 0)
+      (effects (font (size 1.27 1.27)) (justify left) hide)
     )
   )
@@
     )
   )
-  (global_label "AM1" (shape input) (at 142.24 114.3 180) (fields_autoplaced)
-    (effects (font (size 1.27 1.27)) (justify right))
-    (property "Intersheetrefs" "${INTERSHEET_REFS}" (at 136.2389 114.3 0)
-      (effects (font (size 1.27 1.27)) (justify right) hide)
-    )
-  )
-  (global_label "ADC_X" (shape input) (at 118.618 147.066 0) (fields_autoplaced)
-    (effects (font (size 1.27 1.27)) (justify left))
-    (property "Intersheetrefs" "${INTERSHEET_REFS}" (at 127.3295 147.066 0)
-      (effects (font (size 1.27 1.27)) (justify left) hide)
-    )
+  (global_label "AM1" (shape input) (at 118.618 152.146 0) (fields_autoplaced)
+    (effects (font (size 1.27 1.27)) (justify left))
+    (property "Intersheetrefs" "${INTERSHEET_REFS}" (at 124.6191 152.146 0)
+      (effects (font (size 1.27 1.27)) (justify left) hide)
+    )
