File: rescuetruck-main/vootvan.kicad_pcb (KiCad board)
At the start: 2 copper layers, 242.9 x 76.2 mm, 189 parts, among them IC1 W25Q16JVUXIQ, J1 USB-C 2.0 Receptacle, SW2 Reset, U1 AP2112K-3.3, U10 SLSS49E-3, U11 SLSS49E-3, U12 SLSS49E-3, U13 SLSS49E-3, U14 SLSS49E-3, U15 SLSS49E-3, U16 SLSS49E-3, U17 SLSS49E-3, U18 SLSS49E-3, U19 SLSS49E-3, U2 SLSS49E-3, U20 SLSS49E-3, U21 SLSS49E-3, U22 SLSS49E-3, U23 SLSS49E-3, U24 SLSS49E-3, U25 SLSS49E-3, U26 SLSS49E-3, U27 SLSS49E-3, U28 SLSS49E-3, U29 SLSS49E-3, U3 RP2040, U30 SLSS49E-3, U31 SLSS49E-3, U32 SLSS49E-3, U33 SLSS49E-3, U34 SLSS49E-3, U35 SLSS49E-3, U36 SLSS49E-3, U37 SLSS49E-3, U38 SLSS49E-3, U39 SLSS49E-3, U4 SLSS49E-3, U40 SLSS49E-3, U41 SLSS49E-3, U42 SLSS49E-3, U43 SLSS49E-3, U44 SLSS49E-3, U45 SLSS49E-3, U46 74AHCT1G125, U47 SLSS49E-3, U48 SLSS49E-3, U49 SLSS49E-3, U5 SLSS49E-3, U50 SLSS49E-3, U6 SLSS49E-3, U7 SLSS49E-3, U8 SLSS49E-3, U9 SLSS49E-3, Y2 JGHC S3212000181080

Commit message: continue progress
Parts:
- removed ?: , 
- added H6: MountingHole, MountingHole:MountingHole_2.2mm_M2_DIN965_Pad, F.Cu at (76.7, 65.3)
- moved AM1 5.00 mm to (56.9, 40.5)
- moved AM3 5.00 mm to (182.0, 40.5)
- moved C18 1.90 mm to (222.2, 17.5)
Connections:
- net /MCU/OLED_SCL renamed /MCU/GPIO19
- net ADC_Z renamed /MCU/GPIO26_ADC0
- AM2 pad 16: unconnected-(AM2-I15-Pad16) -> K_30
- AM2 pad 17: unconnected-(AM2-I14-Pad17) -> K_41
- AM2 pad 18: unconnected-(AM2-I13-Pad18) -> K_29
- AM2 pad 19: unconnected-(AM2-I12-Pad19) -> K_17
- AM2 pad 2: unconnected-(AM2-I7-Pad2) -> K_8
- AM2 pad 20: unconnected-(AM2-I11-Pad20) -> K_5
- AM2 pad 21: unconnected-(AM2-I10-Pad21) -> K_6
- AM2 pad 22: unconnected-(AM2-I9-Pad22) -> K_18
- AM2 pad 23: unconnected-(AM2-I8-Pad23) -> K_7
- AM2 pad 3: unconnected-(AM2-I6-Pad3) -> K_19
- AM2 pad 4: unconnected-(AM2-I5-Pad4) -> K_20
- AM2 pad 5: unconnected-(AM2-I4-Pad5) -> K_42
- AM2 pad 6: unconnected-(AM2-I3-Pad6) -> K_31
- AM2 pad 7: unconnected-(AM2-I2-Pad7) -> K_9
- AM2 pad 8: unconnected-(AM2-I1-Pad8) -> K_32
- AM2 pad 9: unconnected-(AM2-I0-Pad9) -> K_43
- AM3 pad 16: unconnected-(AM3-I15-Pad16) -> K_33
- AM3 pad 17: unconnected-(AM3-I14-Pad17) -> K_34
- AM3 pad 18: unconnected-(AM3-I13-Pad18) -> K_23
- AM3 pad 19: unconnected-(AM3-I12-Pad19) -> K_44
- AM3 pad 2: unconnected-(AM3-I7-Pad2) -> GND
- AM3 pad 20: unconnected-(AM3-I11-Pad20) -> K_22
- AM3 pad 21: unconnected-(AM3-I10-Pad21) -> K_10
- AM3 pad 22: unconnected-(AM3-I9-Pad22) -> K_11
- AM3 pad 23: unconnected-(AM3-I8-Pad23) -> K_21
- AM3 pad 3: unconnected-(AM3-I6-Pad3) -> K_24
- AM3 pad 4: unconnected-(AM3-I5-Pad4) -> K_12
- AM3 pad 5: unconnected-(AM3-I4-Pad5) -> K_47
- AM3 pad 6: unconnected-(AM3-I3-Pad6) -> K_36
- AM3 pad 7: unconnected-(AM3-I2-Pad7) -> K_46
- AM3 pad 8: unconnected-(AM3-I1-Pad8) -> K_35
- AM3 pad 9: unconnected-(AM3-I0-Pad9) -> K_45
- U14 pad 2: K_9 -> K_10
- U26 pad 2: K_21 -> K_22
- U3 pad 28: /MCU/GPIO17 -> SELECT3
- U3 pad 29: /MCU/OLED_SDA -> SELECT1
- U3 pad 31: /MCU/GPIO20 -> SELECT2
- U3 pad 35: /MCU/GPIO23 -> SELECT0
- U3 pad 37: /MCU/GPIO25 -> AM2
- U3 pad 39: ADC_X -> AM0
- U3 pad 41: /MCU/GPIO29_ADC3 -> AM1
- U3 pad 8: /MCU/GPIO6 -> RGB MCU
- U38 pad 2: K_33 -> K_34
- U50 pad 2: K_45 -> K_46
Routing:
- net +3V3: track 133.8 -> 995.2 mm, vias 48 -> 51
- net AM0: track 0.00 -> 166.0 mm, vias 0 -> 2
- net AM1: track 0.00 -> 101.8 mm, vias 0 -> 2
- net K_45: track 112.9 -> 43.4 mm
- net SELECT3: track 121.6 -> 187.3 mm, vias 3 -> 4
- net K_10: track 0.00 -> 64.9 mm
- net K_46: track 0.00 -> 63.2 mm
- net SELECT2: track 121.8 -> 184.3 mm, vias 3 -> 4
- net SELECT1: track 121.4 -> 181.8 mm, vias 3 -> 4
- net SELECT0: track 122.0 -> 180.4 mm, vias 3 -> 4
- net GND: track 287.1 -> 229.0 mm
- net K_34: track 0.00 -> 56.9 mm
- net K_9: track 110.1 -> 65.5 mm
- net K_33: track 76.3 -> 32.8 mm
- net AM2: track 0.00 -> 41.5 mm
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
Commit message: update
Other:
- board text added: "change the stabs for without ring!!!! MOVE LEDS"
