File: rescuetruck-main/vootvan.kicad_sch (KiCad schematic)
At the start: 242 parts, among them U4 SLSS49E-3, U5 SLSS49E-3

Commit message: deleted caps, res from moon project
Parts:
- removed C17 (x23), C18 (x24), C21 (x23), C22 (x24): 100n, Capacitor_SMD:C_0402_1005Metric, symbol Device:C
- removed R7 (x23), R8 (x24): 10k, Resistor_SMD:R_0402_1005Metric, symbol Device:R
Connections:
- net K_1: now also U5.2 (OUT)
- net K_11: now also U5.2 (OUT)
- net K_12: now also U4.2 (OUT)
- net K_13: now also U5.2 (OUT)
- net K_14: now also U4.2 (OUT)
- net K_15: now also U5.2 (OUT)
- net K_16: now also U4.2 (OUT)
- net K_17: now also U5.2 (OUT)
- net K_18: now also U4.2 (OUT)
- net K_19: now also U5.2 (OUT)
- net K_2: now also U4.2 (OUT)
- net K_20: now also U4.2 (OUT)
- net K_21: now also U5.2 (OUT)
- net K_22: now also U4.2 (OUT)
- net K_23: now also U5.2 (OUT)
- net K_24: now also U4.2 (OUT)
- net K_25: now also U5.2 (OUT)
- net K_26: now also U4.2 (OUT)
- net K_27: now also U5.2 (OUT)
- net K_28: now also U4.2 (OUT)
- net K_29: now also U5.2 (OUT)
- net K_3: now also U5.2 (OUT)
- net K_30: now also U4.2 (OUT)
- net K_31: now also U5.2 (OUT)
- net K_32: now also U4.2 (OUT)
- net K_33: now also U5.2 (OUT)
- net K_34: now also U4.2 (OUT)
- net K_35: now also U5.2 (OUT)
- net K_36: now also U4.2 (OUT)
- net K_37: now also U5.2 (OUT)
- net K_38: now also U4.2 (OUT)
- net K_39: now also U5.2 (OUT)
- net K_4: now also U4.2 (OUT)
- net K_40: now also U4.2 (OUT)
- net K_41: now also U5.2 (OUT)
- net K_42: now also U4.2 (OUT)
- net K_43: now also U5.2 (OUT)
- net K_44: now also U4.2 (OUT)
- net K_45: now also U5.2 (OUT)
- net K_46: now also U4.2 (OUT)
- net K_47: now also U4.2 (OUT)
- net K_5: now also U5.2 (OUT)
- net K_6: now also U4.2 (OUT)
- net K_7: now also U5.2 (OUT)
- net K_8: now also U4.2 (OUT)
- net K_9: now also U5.2 (OUT)
Other:
- moved on the sheet: U4, U5

Commit message: vootvan progress
Parts:
- added H1, H2, H3, H4, H5, H7: MountingHole, Moonpad:MountingHole_2.2mm_M2, symbol Mechanical:MountingHole
Connections:
- net AM0: no longer AM2.1 (COM), AM3.1 (COM)
- net K_1: now also AM1.21 (I10)
- net K_13: now also AM1.20 (I11)
- net K_14: now also AM1.22 (I9)
- net K_15: now also AM1.5 (I4)
- net K_16: now also AM1.2 (I7)
- net K_2: now also AM1.23 (I8)
- net K_21: now also U4.2 (OUT)
- net K_22: no longer U4.2 (OUT)
- net K_25: now also AM1.19 (I12)
- net K_26: now also AM1.17 (I14)
- net K_27: now also AM1.7 (I2)
- net K_28: now also AM1.8 (I1)
- net K_3: now also AM1.3 (I6)
- net K_33: now also U4.2 (OUT)
- net K_34: no longer U4.2 (OUT)
- net K_37: now also AM1.18 (I13)
- net K_38: now also AM1.16 (I15)
- net K_39: now also AM1.9 (I0)
- net K_4: now also AM1.4 (I5)
- net K_40: now also AM1.6 (I3)
- net K_45: now also U4.2 (OUT)
- net K_46: no longer U4.2 (OUT)
- net K_9: now also U4.2 (OUT)
- new net AM1: AM2.1 (COM)
- new net AM2: AM3.1 (COM)
Other:
- moved on the sheet: AM1, AM2

Commit message: continue progress
Parts:
- added H6: MountingHole, MountingHole:MountingHole_2.2mm_M2_DIN965_Pad, symbol Mechanical:MountingHole
Connections:
- net GND: now also AM3.2 (I7)
- net K_10: now also AM3.21 (I10), U4.2 (OUT)
- net K_11: now also AM3.22 (I9)
- net K_12: now also AM3.4 (I5)
- net K_17: now also AM2.19 (I12)
- net K_18: now also AM2.22 (I9)
- net K_19: now also AM2.3 (I6)
- net K_20: now also AM2.4 (I5)
- net K_21: now also AM3.23 (I8); no longer U4.2 (OUT)
- net K_22: now also AM3.20 (I11), U4.2 (OUT)
- net K_23: now also AM3.18 (I13)
- net K_24: now also AM3.3 (I6)
- net K_29: now also AM2.18 (I13)
- net K_30: now also AM2.16 (I15)
- net K_31: now also AM2.6 (I3)
- net K_32: now also AM2.8 (I1)
- net K_33: now also AM3.16 (I15); no longer U4.2 (OUT)
- net K_34: now also AM3.17 (I14), U4.2 (OUT)
- net K_35: now also AM3.8 (I1)
- net K_36: now also AM3.6 (I3)
- net K_41: now also AM2.17 (I14)
- net K_42: now also AM2.5 (I4)
- net K_43: now also AM2.9 (I0)
- net K_44: now also AM3.19 (I12)
- net K_45: now also AM3.9 (I0); no longer U4.2 (OUT)
- net K_46: now also AM3.7 (I2), U4.2 (OUT)
- net K_47: now also AM3.5 (I4)
- net K_5: now also AM2.20 (I11)
- net K_6: now also AM2.21 (I10)
- net K_7: now also AM2.23 (I8)
- net K_8: now also AM2.2 (I7)
- net K_9: now also AM2.7 (I2); no longer U4.2 (OUT)
Other:
- note added: "H6 plated"
- note added: "swapped k44 and k9 to shorten traces"
- moved on the sheet: H1, H2, H3, H4, H5, H7

Commit message: update
Parts:
- S1: footprint PCM_marbastlib-mx:STAB_MX_P_2.75u -> PCM_marbastlib-mx:STAB_MX_2.75u
- S2: footprint PCM_marbastlib-mx:STAB_MX_P_6.25u -> PCM_marbastlib-mx:STAB_MX_6.25u
- S3: footprint PCM_marbastlib-mx:STAB_MX_P_2.25u -> PCM_marbastlib-mx:STAB_MX_2.25u
Changed lines of the file:
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@@
       (effects (font (size 1.27 1.27)) (justify left))
     )
-    (property "Footprint" "PCM_marbastlib-mx:STAB_MX_P_6.25u" (at 172.72 374.904 0)
+    (property "Footprint" "PCM_marbastlib-mx:STAB_MX_6.25u" (at 172.72 374.904 0)
       (effects (font (size 1.27 1.27)) hide)
     )
@@
       (effects (font (size 1.27 1.27)) (justify left))
     )
-    (property "Footprint" "PCM_marbastlib-mx:STAB_MX_P_2.75u" (at 143.51 373.634 0)
+    (property "Footprint" "PCM_marbastlib-mx:STAB_MX_2.75u" (at 143.51 373.634 0)
       (effects (font (size 1.27 1.27)) hide)
     )
@@
       (effects (font (size 1.27 1.27)) (justify left))
     )
-    (property "Footprint" "PCM_marbastlib-mx:STAB_MX_P_2.25u" (at 202.946 374.396 0)
+    (property "Footprint" "PCM_marbastlib-mx:STAB_MX_2.25u" (at 202.946 374.396 0)
       (effects (font (size 1.27 1.27)) hide)
     )
