File: Project/rgb.kicad_sch (KiCad schematic)
At the start: 49 parts, among them U5 74AHCT1G125

Commit message: created production files
Parts:
- D2, D3, D5, D6: value SK6812MINI -> SK6812MINI-E
Changed lines of the file:
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@@
       (effects (font (size 1.27 1.27)))
     )
-    (property "Value" "SK6812MINI" (at 90.678 167.64 0)
+    (property "Value" "SK6812MINI-E" (at 83.058 158.75 0)
       (effects (font (size 1.27 1.27)) hide)
     )
@@
       (effects (font (size 1.27 1.27)))
     )
-    (property "Value" "SK6812MINI" (at 90.932 132.334 0)
+    (property "Value" "SK6812MINI-E" (at 98.552 123.444 0)
       (effects (font (size 1.27 1.27)) hide)
     )
@@
       (effects (font (size 1.27 1.27)))
     )
-    (property "Value" "SK6812MINI" (at 113.538 167.64 0)
+    (property "Value" "SK6812MINI-E" (at 105.918 158.75 0)
       (effects (font (size 1.27 1.27)) hide)
     )
@@
       (effects (font (size 1.27 1.27)))
     )
-    (property "Value" "SK6812MINI" (at 128.778 167.64 0)
+    (property "Value" "SK6812MINI-E" (at 121.158 158.75 0)
       (effects (font (size 1.27 1.27)) hide)
     )
@@
       (effects (font (size 1.27 1.27)))
     )
-    (property "Value" "SK6812MINI" (at 113.792 64.77 0)
+    (property "Value" "SK6812MINI-E" (at 121.412 55.88 0)
       (effects (font (size 1.27 1.27)) hide)
     )
@@
       (effects (font (size 1.27 1.27)))
     )
-    (property "Value" "SK6812MINI" (at 75.438 98.044 0)
+    (property "Value" "SK6812MINI-E" (at 67.818 89.154 0)
       (effects (font (size 1.27 1.27)) hide)
     )
@@
       (effects (font (size 1.27 1.27)))
     )
-    (property "Value" "SK6812MINI" (at 202.692 132.334 0)
+    (property "Value" "SK6812MINI-E" (at 210.312 123.444 0)
       (effects (font (size 1.27 1.27)) hide)
     )
@@
       (effects (font (size 1.27 1.27)))
     )
-    (property "Value" "SK6812MINI" (at 113.792 132.334 0)
+    (property "Value" "SK6812MINI-E" (at 121.412 123.444 0)
       (effects (font (size 1.27 1.27)) hide)
     )
@@
       (effects (font (size 1.27 1.27)))
     )
-    (property "Value" "SK6812MINI" (at 113.538 98.044 0)
+    (property "Value" "SK6812MINI-E" (at 105.918 89.154 0)
       (effects (font (size 1.27 1.27)) hide)
     )
@@
       (effects (font (size 1.27 1.27)))
     )
-    (property "Value" "SK6812MINI" (at 240.792 64.77 0)
+    (property "Value" "SK6812MINI-E" (at 248.412 55.88 0)
       (effects (font (size 1.27 1.27)) hide)
     )
@@
       (effects (font (size 1.27 1.27)))
     )
-    (property "Value" "SK6812MINI" (at 75.692 67.056 0)
+    (property "Value" "SK6812MINI-E" (at 83.312 55.88 0)
       (effects (font (size 1.27 1.27)) hide)
     )
@@
       (effects (font (size 1.27 1.27)))
     )
-    (property "Value" "SK6812MINI" (at 129.032 132.334 0)
+    (property "Value" "SK6812MINI-E" (at 136.652 123.444 0)
       (effects (font (size 1.27 1.27)) hide)
     )
@@
       (effects (font (size 1.27 1.27)))
     )
-    (property "Value" "SK6812MINI" (at 240.792 132.334 0)
+    (property "Value" "SK6812MINI-E" (at 248.412 123.444 0)
       (effects (font (size 1.27 1.27)) hide)
     )
@@
       (effects (font (size 1.27 1.27)))
     )
-    (property "Value" "SK6812MINI" (at 75.692 132.334 0)
+    (property "Value" "SK6812MINI-E" (at 83.312 123.444 0)
       (effects (font (size 1.27 1.27)) hide)
     )
@@
       (effects (font (size 1.27 1.27)))
     )
-    (property "Value" "SK6812MINI" (at 202.438 167.64 0)
+    (property "Value" "SK6812MINI-E" (at 194.818 158.75 0)
       (effects (font (size 1.27 1.27)) hide)
     )
@@
       (effects (font (size 1.27 1.27)))
     )
-    (property "Value" "SK6812MINI" (at 90.678 98.044 0)
+    (property "Value" "SK6812MINI-E" (at 83.058 89.154 0)
       (effects (font (size 1.27 1.27)) hide)
     )
@@
       (effects (font (size 1.27 1.27)))
     )
-    (property "Value" "SK6812MINI" (at 90.932 67.056 0)
+    (property "Value" "SK6812MINI-E" (at 98.552 55.88 0)
       (effects (font (size 1.27 1.27)) hide)
     )
@@
       (effects (font (size 1.27 1.27)))
     )
-    (property "Value" "SK6812MINI" (at 75.438 167.64 0)
+    (property "Value" "SK6812MINI-E" (at 67.818 158.75 0)
       (effects (font (size 1.27 1.27)) hide)
     )
@@
       (effects (font (size 1.27 1.27)))
     )
-    (property "Value" "SK6812MINI" (at 225.552 132.334 0)
+    (property "Value" "SK6812MINI-E" (at 233.172 123.444 0)
       (effects (font (size 1.27 1.27)) hide)
     )
@@
       (effects (font (size 1.27 1.27)))
     )
-    (property "Value" "SK6812MINI" (at 187.452 64.77 0)
+    (property "Value" "SK6812MINI-E" (at 195.072 55.88 0)
       (effects (font (size 1.27 1.27)) hide)
     )
@@
       (effects (font (size 1.27 1.27)))
     )
-    (property "Value" "SK6812MINI" (at 128.778 98.044 0)
+    (property "Value" "SK6812MINI-E" (at 121.158 89.154 0)
       (effects (font (size 1.27 1.27)) hide)
     )
@@
       (effects (font (size 1.27 1.27)))
     )
-    (property "Value" "SK6812MINI" (at 240.538 167.64 0)
+    (property "Value" "SK6812MINI-E" (at 232.918 158.75 0)
       (effects (font (size 1.27 1.27)) hide)
     )
@@
       (effects (font (size 1.27 1.27)))
     )
-    (property "Value" "SK6812MINI" (at 187.198 167.64 0)
+    (property "Value" "SK6812MINI-E" (at 179.578 158.75 0)
       (effects (font (size 1.27 1.27)) hide)
     )
@@
       (effects (font (size 1.27 1.27)))
     )
-    (property "Value" "SK6812MINI" (at 225.552 64.77 0)
+    (property "Value" "SK6812MINI-E" (at 233.172 55.88 0)
       (effects (font (size 1.27 1.27)) hide)
     )
@@
       (effects (font (size 1.27 1.27)))
     )
-    (property "Value" "SK6812MINI" (at 225.298 98.044 0)
+    (property "Value" "SK6812MINI-E" (at 217.678 89.154 0)
       (effects (font (size 1.27 1.27)) hide)
     )
@@
       (effects (font (size 1.27 1.27)))
     )
-    (property "Value" "SK6812MINI" (at 225.298 167.64 0)
+    (property "Value" "SK6812MINI-E" (at 217.678 158.75 0)
       (effects (font (size 1.27 1.27)) hide)
     )
@@
       (effects (font (size 1.27 1.27)))
     )
-    (property "Value" "SK6812MINI" (at 240.538 98.044 0)
+    (property "Value" "SK6812MINI-E" (at 232.918 89.154 0)
       (effects (font (size 1.27 1.27)) hide)
     )
@@
       (effects (font (size 1.27 1.27)))
     )
-    (property "Value" "SK6812MINI" (at 202.692 64.77 0)
+    (property "Value" "SK6812MINI-E" (at 210.312 55.88 0)
       (effects (font (size 1.27 1.27)) hide)
     )
@@
       (effects (font (size 1.27 1.27)))
     )
-    (property "Value" "SK6812MINI" (at 187.198 98.044 0)
+    (property "Value" "SK6812MINI-E" (at 179.578 89.154 0)
       (effects (font (size 1.27 1.27)) hide)
     )
@@
       (effects (font (size 1.27 1.27)))
     )
-    (property "Value" "SK6812MINI" (at 129.032 64.77 0)
+    (property "Value" "SK6812MINI-E" (at 136.652 55.88 0)
       (effects (font (size 1.27 1.27)) hide)
     )
@@
       (effects (font (size 1.27 1.27)))
     )
-    (property "Value" "SK6812MINI" (at 202.438 98.044 0)
+    (property "Value" "SK6812MINI-E" (at 194.818 89.154 0)
       (effects (font (size 1.27 1.27)) hide)
     )
@@
       (effects (font (size 1.27 1.27)))
     )
-    (property "Value" "SK6812MINI" (at 187.452 132.334 0)
+    (property "Value" "SK6812MINI-E" (at 195.072 123.444 0)
       (effects (font (size 1.27 1.27)) hide)
     )
@@
       (effects (font (size 1.27 1.27)))
     )
-    (property "Value" "SK6812MINI-E" (at 60.452 67.056 0)
+    (property "Value" "SK6812MINI-E" (at 68.072 55.88 0)
       (effects (font (size 1.27 1.27)) hide)
     )
