File: Project/rgb VAN.kicad_sch (KiCad schematic)
At the start: 49 parts, among them U5 74AHCT1G125

Commit message: rgb footprints changed, fresh gerbers, production
Parts:
- D1, D2, D3, D4, D5, D6: footprint PCM_marbastlib-various:LED_6028R -> cipulot_parts:SK6812-MINI-E; symbol PCM_marbastlib-various:SK6812MINI-E -> cipulot_parts:YS-SK6812MINI-E
Connections:
- net GND: now also D1.3 (VSS), D1.3 (VSS), D1.3 (VSS), D1.3 (VSS), D1.3 (VSS), D1.3 (VSS), D1.3 (VSS), D1.3 (VSS), D2.3 (VSS), D2.3 (VSS), D2.3 (VSS), D2.3 (VSS), D2.3 (VSS), D2.3 (VSS), D2.3 (VSS), D2.3 (VSS), D3.3 (VSS), D3.3 (VSS), D3.3 (VSS), D3.3 (VSS), D3.3 (VSS), D3.3 (VSS), D3.3 (VSS), D3.3 (VSS), D4.3 (VSS), D4.3 (VSS), D4.3 (VSS), D4.3 (VSS), D4.3 (VSS), D4.3 (VSS), D4.3 (VSS), D5.3 (VSS), D5.3 (VSS), D5.3 (VSS), D5.3 (VSS), D5.3 (VSS), D5.3 (VSS), D5.3 (VSS), D5.3 (VSS), D6.3 (VSS), D6.3 (VSS), D6.3 (VSS), D6.3 (VSS), D6.3 (VSS), D6.3 (VSS), D6.3 (VSS), D6.3 (VSS); no longer D1.4 (VSS), D1.4 (VSS), D1.4 (VSS), D1.4 (VSS), D1.4 (VSS), D1.4 (VSS), D1.4 (VSS), D1.4 (VSS), D2.4 (VSS), D2.4 (VSS), D2.4 (VSS), D2.4 (VSS), D2.4 (VSS), D2.4 (VSS), D2.4 (VSS), D2.4 (VSS), D3.4 (VSS), D3.4 (VSS), D3.4 (VSS), D3.4 (VSS), D3.4 (VSS), D3.4 (VSS), D3.4 (VSS), D3.4 (VSS), D4.4 (VSS), D4.4 (VSS), D4.4 (VSS), D4.4 (VSS), D4.4 (VSS), D4.4 (VSS), D4.4 (VSS), D5.4 (VSS), D5.4 (VSS), D5.4 (VSS), D5.4 (VSS), D5.4 (VSS), D5.4 (VSS), D5.4 (VSS), D5.4 (VSS), D6.4 (VSS), D6.4 (VSS), D6.4 (VSS), D6.4 (VSS), D6.4 (VSS), D6.4 (VSS), D6.4 (VSS), D6.4 (VSS)
- net RGB: now also D4.4 (DIN); no longer D4.3 (DIN)
- net at D4.2 (DOUT): now also D6.4 (DIN); no longer D6.3 (DIN) (x6)
- net at D1.2 (DOUT): now also D4.4 (DIN); no longer D4.3 (DIN) (x6)
- net at D3.2 (DOUT): now also D2.4 (DIN); no longer D2.3 (DIN) (x8)
- net at D5.2 (DOUT): now also D3.4 (DIN); no longer D3.3 (DIN) (x8)
- net at D6.2 (DOUT): now also D5.4 (DIN); no longer D5.3 (DIN) (x8)
- net at D1.2 (DOUT): now also D6.4 (DIN); no longer D6.3 (DIN) (x2)
- net at D2.2 (DOUT): now also D1.4 (DIN); no longer D1.3 (DIN) (x7)
- net at D4.2 (DOUT): now also D1.4 (DIN); no longer D1.3 (DIN)
