File: Project/vootington V4N.kicad_sch (KiCad schematic)
At the start: 134 parts, among them U4 SLSS49E-3, U5 SLSS49E-3

Commit message: update
Parts:
- renumbered H5 to H2, H2 to H3, H6 to H4, H3 to H5, H7 to H6, H4 to H7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
