File: Project/vootington V4N V2.kicad_pcb (KiCad board)
At the start: 2 copper layers, 242.9 x 95.2 mm, 339 parts, among them J1 Conn_01x04, J10 Conn_01x01, J11 Conn_01x01, J12 USB_C sink board 1.3mm, J13 JST SH, J14 Pico EZmate, J2 Conn_01x01, J3 Conn_01x01, J4 Conn_01x01, J5 Conn_01x01, J6 Conn_01x01, J7 Conn_01x01, J8 Conn_01x01, J9 Conn_01x01, SW1 SKQGABE010, SW2 SKQGABE010, U1 SLSS49E-3, U10 SLSS49E-3, U11 SLSS49E-3, U12 SLSS49E-3, U13 SLSS49E-3, U14 SLSS49E-3, U15 SLSS49E-3, U16 SLSS49E-3, U17 SLSS49E-3, U18 SLSS49E-3, U19 SLSS49E-3, U2 SLSS49E-3, U20 SLSS49E-3, U21 SLSS49E-3, U22 SLSS49E-3, U23 SLSS49E-3, U24 SLSS49E-3, U25 SLSS49E-3, U26 SLSS49E-3, U27 SLSS49E-3, U28 SLSS49E-3, U29 SLSS49E-3, U3 SLSS49E-3, U30 SLSS49E-3, U31 SLSS49E-3, U32 SLSS49E-3, U33 SLSS49E-3, U34 SLSS49E-3, U35 SLSS49E-3, U36 SLSS49E-3, U37 SLSS49E-3, U38 SLSS49E-3, U39 SLSS49E-3, U4 SLSS49E-3, U40 SLSS49E-3, U41 SLSS49E-3, U42 SLSS49E-3, U43 SLSS49E-3, U44 SLSS49E-3, U45 SLSS49E-3, U46 SLSS49E-3, U47 SLSS49E-3, U48 SLSS49E-3, U49 SLSS49E-3, U5 SLSS49E-3, U50 SLSS49E-3, U51 SLSS49E-3, U52 SLSS49E-3, U53 STM32F072CBT6, U54 XC6206PxxxMR-Regulator_Linear, U55 PRTR5V0U2X, U56 74AHCT1G125, U57 74HC4051, U58 74HC4051, U59 74HC4051, U6 SLSS49E-3, U60 74HC4051, U61 74HC4051, U62 74HC4051, U63 74HC4051, U64 AP2112K-3.3, U7 SLSS49E-3, U8 SLSS49E-3, U9 SLSS49E-3

Commit message: backup
Parts:
- moved C44 0.41 mm to (60.3, 96.0)
Routing:
- net GND: track 294.3 -> 296.9 mm, vias 185 -> 187
Changed lines of the file:
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@@
 		(fp_arc
 			(start 15.28125 7.500001)
-			(mid 15.1348 7.853536)
+			(mid 15.134806 7.853571)
 			(end 14.78125 8.000001)
 			(stroke
@@
 		(fp_arc
 			(start 14.780039 -5.999999)
-			(mid 15.133602 -5.853545)
+			(mid 15.133567 -5.853539)
 			(end 15.280039 -5.499999)
 			(stroke
@@
 		(fp_arc
 			(start 9.03125 8.000001)
-			(mid 8.677693 7.853543)
+			(mid 8.677729 7.853537)
 			(end 8.53125 7.500001)
 			(stroke
@@
 		(fp_arc
 			(start 53.38125 7.500001)
-			(mid 53.2348 7.853536)
+			(mid 53.234806 7.853571)
 			(end 52.88125 8.000001)
 			(stroke
@@
 		(fp_arc
 			(start 52.880039 -5.999999)
-			(mid 53.233602 -5.853545)
+			(mid 53.233567 -5.853539)
 			(end 53.380039 -5.499999)
 			(stroke
@@
 		(fp_arc
 			(start 47.13125 8.000001)
-			(mid 46.777693 7.853543)
+			(mid 46.777729 7.853537)
 			(end 46.63125 7.500001)
 			(stroke
@@
 		(fp_arc
 			(start 46.63125 -5.499999)
-			(mid 46.777699 -5.853535)
+			(mid 46.777693 -5.853571)
 			(end 47.13125 -5.999999)
 			(stroke
@@
 		(fp_arc
 			(start 15.28125 7.500001)
-			(mid 15.1348 7.853536)
+			(mid 15.134806 7.853571)
 			(end 14.78125 8.000001)
 			(stroke
@@
 		(fp_arc
 			(start 14.780039 -5.999999)
-			(mid 15.133602 -5.853545)
+			(mid 15.133567 -5.853539)
 			(end 15.280039 -5.499999)
 			(stroke
@@
 		(fp_arc
 			(start 9.03125 8.000001)
-			(mid 8.677693 7.853543)
+			(mid 8.677729 7.853537)
 			(end 8.53125 7.500001)
 			(stroke
@@
 	(footprint "Capacitor_SMD:C_0402_1005Metric"
 		(layer "B.Cu")
-		(at 60.325 95.6325 180)
+		(at 60.325 96.04375 180)
 		(descr "Capacitor SMD 0402 (1005 Metric), square (rectangular) end terminal, IPC_7351 nominal, (Body size source: IPC-SM-782 page 76, https://www.pcb-3d.com/wordpress/wp-content/uploads/ipc-sm-782a_amendment_1_and_2.pdf), generated with kicad-footprint-generator")
 		(tags "capacitor")
@@
 	)
 	(via
+		(at 86.002262 69.91875)
+		(size 0.8)
+		(drill 0.4)
+		(layers "F.Cu" "B.Cu")
+		(net 2)
+	)
+	(via
 		(at 86.51875 79.375)
 		(size 0.8)
@@
 	)
 	(via
+		(at 165.1 71.4375)
+		(size 0.8)
+		(drill 0.4)
+		(layers "F.Cu" "B.Cu")
+		(net 2)
+	)
+	(via
 		(at 36.5125 98.425)
 		(size 0.8)
@@
 	)
 	(segment
+		(start 86.03875 71.4375)
+		(end 86.03875 69.955238)
+		(width 0.25)
+		(layer "B.Cu")
+		(net 2)
+	)
+	(segment
 		(start 60.919654 26.570992)
 		(end 60.907654 26.582992)
@@
 	)
 	(segment
+		(start 86.03875 69.955238)
+		(end 86.002262 69.91875)
+		(width 0.25)
+		(layer "B.Cu")
+		(net 2)
+	)
+	(segment
 		(start 227.557463 64.650224)
 		(end 227.545463 64.662224)
@@
 		(layer "B.Cu")
 		(net 2)
+	)
+	(segment
+		(start 166.2075 71.4375)
+		(end 165.1 71.4375)
+		(width 0.25)
+		(layer "B.Cu")
+		(net 2)

Commit message: update
Parts:
- moved C66 0.31 mm to (33.3, 31.0)
Routing:
- net GND: track 296.9 -> 326.9 mm, vias 187 -> 190
- net +5V: track 1311.3 -> 1308.0 mm
- net RGB: track 8.32 -> 7.75 mm
Changed lines of the file:
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@@
 	(footprint "Capacitor_SMD:C_0402_1005Metric"
 		(layer "B.Cu")
-		(at 33.65125 30.95625)
+		(at 33.3375 30.95625)
 		(descr "Capacitor SMD 0402 (1005 Metric), square (rectangular) end terminal, IPC_7351 nominal, (Body size source: IPC-SM-782 page 76, https://www.pcb-3d.com/wordpress/wp-content/uploads/ipc-sm-782a_amendment_1_and_2.pdf), generated with kicad-footprint-generator")
 		(tags "capacitor")
@@
 	)
 	(segment
-		(start 30.725044 32.54375)
-		(end 30.725044 29.599956)
-		(width 0.25)
-		(layer "F.Cu")
-		(net 1)
-	)
-	(segment
 		(start 60.332837 29.376587)
 		(end 60.325 29.36875)
@@
 	)
 	(segment
-		(start 30.98025 29.34475)
-		(end 34.98125 29.34475)
+		(start 31.66575 44.45)
+		(end 32.54375 44.45)
 		(width 0.25)
 		(layer "F.Cu")
@@
 	)
 	(segment
-		(start 31.66575 44.45)
-		(end 32.54375 44.45)
+		(start 30.872 66.675)
+		(end 30.872 45.24375)
 		(width 0.25)
 		(layer "F.Cu")
@@
 	)
 	(segment
-		(start 30.872 66.675)
-		(end 30.872 45.24375)
+		(start 33.924044 29.34475)
+		(end 34.98125 29.34475)
 		(width 0.25)
 		(layer "F.Cu")
@@
 	)
 	(segment
+		(start 30.725044 32.54375)
+		(end 33.924044 29.34475)
+		(width 0.25)
+		(layer "F.Cu")
+		(net 1)
+	)
+	(segment
 		(start 51.59375 25.4)
 		(end 50.149853 25.4)
@@
 		(net 1)
 	)
-	(segment
-		(start 30.725044 29.599956)
-		(end 30.98025 29.34475)
-		(width 0.25)
-		(layer "F.Cu")
-		(net 1)
-	)
 	(via
 		(at 65.88125 82.55)
@@
 	)
 	(segment
-		(start 34.13125 30.95625)
-		(end 34.13125 29.6825)
-		(width 0.25)
-		(layer "B.Cu")
-		(net 1)
-	)
-	(segment
 		(start 139.38625 67.46875)
 		(end 140.49375 67.46875)
@@
 	)
 	(segment
+		(start 33.8175 29.36875)
+		(end 33.8175 30.95625)
+		(width 0.381)
+		(layer "B.Cu")
+		(net 1)
+	)
+	(segment
 		(start 215.58625 67.46875)
 		(end 216.69375 67.46875)
@@
 	)
 	(segment
-		(start 34.13125 30.95625)
-		(end 34.13125 32.85925)
-		(width 0.25)
-		(layer "B.Cu")
-		(net 1)
-	)
-	(segment
 		(start 162.23875 83.41775)
 		(end 162.23875 82.55)
@@
 	)
 	(segment
+		(start 29.558052 29.36875)
+		(end 28.575 28.385698)
+		(width 0.25)
+		(layer "F.Cu")
+		(net 2)
+	)
+	(segment
 		(start 41.275 48.73625)
 		(end 41.275 47.6885)
@@
 	)
 	(segment
+		(start 30.1625 23.8125)
+		(end 30.95625 23.8125)
+		(width 0.25)
+		(layer "F.Cu")
+		(net 2)
+	)
+	(segment
+		(start 28.575 19.84375)
+		(end 30.1625 18.25625)
+		(width 0.25)
+		(layer "F.Cu")
+		(net 2)
+	)
+	(segment
+		(start 30.95625 29.36875)
+		(end 30.95625 30.1625)
+		(width 0.25)
+		(layer "F.Cu")
+		(net 2)
+	)
+	(segment
+		(start 28.575 25.4)
+		(end 30.1625 23.8125)
+		(width 0.25)
+		(layer "F.Cu")
+		(net 2)
+	)
+	(segment
 		(start 57.039177 22.429988)
 		(end 57.0495 22.440311)
@@
 	)
 	(segment
+		(start 28.575 28.385698)
+		(end 28.575 25.4)
+		(width 0.25)
+		(layer "F.Cu")
+		(net 2)
+	)
+	(segment
 		(start 53.727246 22.429988)
 		(end 57.039177 22.429988)
@@
 		(net 2)
 	)
+	(segment
+		(start 30.1625 18.25625)
+		(end 30.95625 18.25625)
+		(width 0.25)
+		(layer "F.Cu")
+		(net 2)
+	)
+	(segment
+		(start 30.95625 29.36875)
+		(end 29.558052 29.36875)
+		(width 0.25)
+		(layer "F.Cu")
+		(net 2)
+	)
+	(segment
+		(start 28.575 14.2875)
+		(end 28.575 25.4)
+		(width 0.25)
+		(layer "F.Cu")
+		(net 2)
+	)
 	(via
 		(at 34.13125 41.275)
@@
 	)
 	(via
+		(at 30.95625 23.8125)
+		(size 0.8)
+		(drill 0.4)
+		(layers "F.Cu" "B.Cu")
+		(net 2)
+	)
+	(via
 		(at 124.61875 79.375)
 		(size 0.8)
@@
 	)
 	(via
+		(at 30.95625 29.36875)
+		(size 0.8)
+		(drill 0.4)
+		(layers "F.Cu" "B.Cu")
+		(net 2)
+	)
+	(via
 		(at 115.09375 60.325)
 		(size 0.8)
@@
 	)
 	(via
+		(at 30.95625 18.25625)
+		(size 0.8)
+		(drill 0.4)
+		(layers "F.Cu" "B.Cu")
+		(net 2)
+	)
+	(via
 		(at 181.76875 79.375)
 		(size 0.8)
@@
 	)
 	(via
+		(at 30.95625 30.1625)
+		(size 0.8)
+		(drill 0.4)
+		(layers "F.Cu" "B.Cu")
+		(net 2)
+	)
+	(via
 		(at 162.71875 79.375)
 		(size 0.8)
@@
 	)
 	(via
-		(at 33.161691 30.09325)
-		(size 0.8)
-		(drill 0.4)
-		(layers "F.Cu" "B.Cu")
-		(net 2)
-	)
-	(via
 		(at 257.39725 47.117)
 		(size 0.8)
@@
 	)
 	(segment
+		(start 32.8575 23.8125)
+		(end 30.95625 23.8125)
+		(width 0.25)
+		(layer "B.Cu")
+		(net 2)
+	)
+	(segment
 		(start 51.179 17.420625)
 		(end 51.179 13.3905)
@@
 	)
 	(segment
+		(start 32.8575 29.36875)
+		(end 30.95625 29.36875)
+		(width 0.25)
+		(layer "B.Cu")
+		(net 2)
+	)
+	(segment
 		(start 110.675 85.229)
 		(end 112.129 85.229)
@@
 	)
 	(segment
+		(start 32.8575 18.25625)
+		(end 30.95625 18.25625)
+		(width 0.25)
+		(layer "B.Cu")
+		(net 2)
+	)
+	(segment
 		(start 190.965106 64.721776)
 		(end 189.511106 64.721776)
@@
 	)
 	(segment
+		(start 32.8575 30.95625)
+		(end 32.06375 30.1625)
+		(width 0.25)
+		(layer "B.Cu")
+		(net 2)
+	)
+	(segment
 		(start 86.03875 71.4375)
 		(end 86.03875 69.955238)
@@
 	)
 	(segment
+		(start 32.06375 30.1625)
+		(end 30.95625 30.1625)
+		(width 0.25)
+		(layer "B.Cu")
+		(net 2)
+	)
+	(segment
 		(start 168.902206 72.193675)
 		(end 170.618675 72.193675)
@@
 	)
 	(segment
-		(start 33.17125 30.95625)
-		(end 33.17125 30.102809)
-		(width 0.381)
-		(layer "B.Cu")
-		(net 2)
-	)
-	(segment
-		(start 33.17125 30.102809)
-		(end 33.161691 30.09325)
-		(width 0.381)
-		(layer "B.Cu")
-		(net 2)
-	)
-	(segment
 		(start 138.557505 26.563155)
 		(end 137.103505 26.563155)
@@
 	)
 	(segment
-		(start 32.8575 29.789059)
-		(end 33.161691 30.09325)
-		(width 0.381)
-		(layer "B.Cu")
-		(net 2)
-	)
-	(segment
 		(start 34.09325 35.17225)
 		(end 34.09325 36.152616)
@@
 	)
 	(segment
-		(start 32.8575 29.36875)
-		(end 32.8575 29.789059)
-		(width 0.381)
-		(layer "B.Cu")
-		(net 2)
-	)
-	(segment
 		(start 131.988386 76.090035)
 		(end 131.988386 77.284982)
@@
 	)
 	(segment
-		(start 32.19325 32.89725)
-		(end 32.19325 29.812)
+		(start 28.694861 31.04396)
+		(end 28.591076 30.940174)
+		(width 0.25)
+		(layer "B.Cu")
+		(net 72)
+	)
+	(segment
+		(start 32.194861 32.91646)
+		(end 32.194861 32.25646)
 		(width 0.25)
 		(layer "B.Cu")
@@
 	)
 	(segment
-		(start 31.75 29.36875)
-		(end 28.575 29.36875)
+		(start 28.591076 30.940174)
+		(end 28.4625 30.811598)
 		(width 0.25)
 		(layer "B.Cu")
@@
 	)
 	(segment
-		(start 32.19325 29.812)
-		(end 31.75 29.36875)
+		(start 28.4625 30.811598)
+		(end 28.4625 28.055)
 		(width 0.25)
 		(layer "B.Cu")
@@
 	)
 	(segment
-		(start 28.2875 29.08125)
-		(end 28.2875 28.055)
+		(start 28.694861 31.04396)
+		(end 30.982361 31.04396)
 		(width 0.25)
 		(layer "B.Cu")
@@
 	)
 	(segment
-		(start 28.575 29.36875)
-		(end 28.2875 29.08125)
+		(start 32.194861 32.25646)
+		(end 30.982361 31.04396)
 		(width 0.25)
 		(layer "B.Cu")

Commit message: revision work
Routing:
- net K_38: track 23.8 -> 19.7 mm
- net K_26: track 16.8 -> 14.3 mm
Changed lines of the file:
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@@
 		(fp_arc
 			(start 15.28125 7.500001)
-			(mid 15.134806 7.853571)
+			(mid 15.1348 7.853536)
 			(end 14.78125 8.000001)
 			(stroke
@@
 		(fp_arc
 			(start 14.780039 -5.999999)
-			(mid 15.133567 -5.853539)
+			(mid 15.133602 -5.853545)
 			(end 15.280039 -5.499999)
 			(stroke
@@
 		(fp_arc
 			(start 9.03125 8.000001)
-			(mid 8.677729 7.853537)
+			(mid 8.677693 7.853543)
 			(end 8.53125 7.500001)
 			(stroke
@@
 		(fp_arc
 			(start 53.38125 7.500001)
-			(mid 53.234806 7.853571)
+			(mid 53.2348 7.853536)
 			(end 52.88125 8.000001)
 			(stroke
@@
 		(fp_arc
 			(start 52.880039 -5.999999)
-			(mid 53.233567 -5.853539)
+			(mid 53.233602 -5.853545)
 			(end 53.380039 -5.499999)
 			(stroke
@@
 		(fp_arc
 			(start 47.13125 8.000001)
-			(mid 46.777729 7.853537)
+			(mid 46.777693 7.853543)
 			(end 46.63125 7.500001)
 			(stroke
@@
 		(fp_arc
 			(start 46.63125 -5.499999)
-			(mid 46.777693 -5.853571)
+			(mid 46.777699 -5.853535)
 			(end 47.13125 -5.999999)
 			(stroke
@@
 		(fp_arc
 			(start 15.28125 7.500001)
-			(mid 15.134806 7.853571)
+			(mid 15.1348 7.853536)
 			(end 14.78125 8.000001)
 			(stroke
@@
 		(fp_arc
 			(start 14.780039 -5.999999)
-			(mid 15.133567 -5.853539)
+			(mid 15.133602 -5.853545)
 			(end 15.280039 -5.499999)
 			(stroke
@@
 		(fp_arc
 			(start 9.03125 8.000001)
-			(mid 8.677729 7.853537)
+			(mid 8.677693 7.853543)
 			(end 8.53125 7.500001)
 			(stroke
@@
 	)
 	(segment
-		(start 71.85 79.2625)
-		(end 71.85 76.73992)
-		(width 0.25)
-		(layer "B.Cu")
-		(net 40)
-	)
-	(segment
 		(start 70.7875 80.325)
 		(end 71.85 79.2625)
@@
 	)
 	(segment
-		(start 71.653125 76.415625)
-		(end 68.73367 73.49617)
-		(width 0.25)
-		(layer "B.Cu")
-		(net 51)
-	)
-	(segment
