File: Project/vootington V4N V2.kicad_pcb (KiCad board)
At the start: 2 copper layers, 242.9 x 95.2 mm, 339 parts, among them J1 Conn_01x04, J10 Conn_01x01, J11 Conn_01x01, J12 USB_C sink board 1.3mm, J13 JST SH, J14 Pico EZmate, J2 Conn_01x01, J3 Conn_01x01, J4 Conn_01x01, J5 Conn_01x01, J6 Conn_01x01, J7 Conn_01x01, J8 Conn_01x01, J9 Conn_01x01, SW1 SKQGABE010, SW2 SKQGABE010, U1 SLSS49E-3, U10 SLSS49E-3, U11 SLSS49E-3, U12 SLSS49E-3, U13 SLSS49E-3, U14 SLSS49E-3, U15 SLSS49E-3, U16 SLSS49E-3, U17 SLSS49E-3, U18 SLSS49E-3, U19 SLSS49E-3, U2 SLSS49E-3, U20 SLSS49E-3, U21 SLSS49E-3, U22 SLSS49E-3, U23 SLSS49E-3, U24 SLSS49E-3, U25 SLSS49E-3, U26 SLSS49E-3, U27 SLSS49E-3, U28 SLSS49E-3, U29 SLSS49E-3, U3 SLSS49E-3, U30 SLSS49E-3, U31 SLSS49E-3, U32 SLSS49E-3, U33 SLSS49E-3, U34 SLSS49E-3, U35 SLSS49E-3, U36 SLSS49E-3, U37 SLSS49E-3, U38 SLSS49E-3, U39 SLSS49E-3, U4 SLSS49E-3, U40 SLSS49E-3, U41 SLSS49E-3, U42 SLSS49E-3, U43 SLSS49E-3, U44 SLSS49E-3, U45 SLSS49E-3, U46 SLSS49E-3, U47 SLSS49E-3, U48 SLSS49E-3, U49 SLSS49E-3, U5 SLSS49E-3, U50 SLSS49E-3, U51 SLSS49E-3, U52 SLSS49E-3, U53 STM32F072CBT6, U54 XC6206PxxxMR-Regulator_Linear, U55 PRTR5V0U2X, U56 74AHCT1G125, U57 74HC4051, U58 74HC4051, U59 74HC4051, U6 SLSS49E-3, U60 74HC4051, U61 74HC4051, U62 74HC4051, U63 74HC4051, U64 AP2112K-3.3, U7 SLSS49E-3, U8 SLSS49E-3, U9 SLSS49E-3

Commit message: wip
Parts:
- added C126: 100nF, Capacitor_SMD:C_0402_1005Metric, B.Cu at (56.5, 55.8)
- added C127: 10nF, Capacitor_SMD:C_0402_1005Metric, B.Cu at (56.5, 53.4)
- added C128: 1uF, Capacitor_SMD:C_0402_1005Metric, B.Cu at (56.5, 52.4)
- added FB1: 1k OHM 100mhz, Fuse:Fuse_0402_1005Metric, B.Cu at (56.5, 54.8)
- added U65: STM32G0B1CBTx, Package_QFP:LQFP-48_7x7mm_P0.5mm, B.Cu at (49.2, 54.8)
- moved U53 33.1 mm to (16.1, 55.0)
- moved C56 2.15 mm to (56.3, 58.2)
- moved C59 2.15 mm to (56.4, 57.1)
- moved C119 0.79 mm to (240.5, 71.4)
- moved C122 0.79 mm to (123.0, 71.4)
- moved C123 0.79 mm to (85.7, 71.4)
- moved C120 0.79 mm to (201.6, 71.4)
- moved C121 0.79 mm to (165.9, 71.4)
- moved C125 0.59 mm to (87.3, 31.0)
- moved C124 0.59 mm to (46.2, 71.4)
Routing:
- net +3V3: track 1091.5 -> 261.7 mm, vias 57 -> 64
- net K_50: track 29.2 -> 14.7 mm
- net NRST: track 16.4 -> 9.04 mm
- net +5V: track 1308.0 -> 1311.7 mm
- net ADC4: track 53.7 -> 55.8 mm
- net GND: track 326.9 -> 328.6 mm
- added copper zone on F.Cu, net +3V3
- added copper zone on B.Cu, net GND
- removed copper zone on F.Cu, net GND
