File: Project/multi V4N.kicad_sch (KiCad schematic)
At the start: 7 parts, among them U4 74HC4051, U6 74HC4051

Commit message: revision work
Parts:
- added C119, C120, C121, C122, C123, C124, C125: 100pF, Capacitor_SMD:C_0402_1005Metric, symbol Device:C_Small
Connections:
- net +3V3: now also C119.1, C120.1, C121.1, C122.1, C123.1, C124.1, C125.1
- net GND: now also C119.2, C120.2, C121.2, C122.2, C123.2, C124.2, C125.2

Commit message: backups
Parts:
- renumbered C119 to C118, C120 to C119, C121 to C120, C122 to C121, C123 to C122, C124 to C123, C125 to C124
Changed lines of the file:
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@@
 			(project "vootington V4N"
 				(path "/7fa06d8b-464b-4050-a0fd-d319cc509390/18fa9a6d-388b-4829-a409-257b50720dd4"
-					(reference "#PWR0363")
+					(reference "#PWR0365")
 					(unit 1)
 				)
@@
 			(project "vootington V4N"
 				(path "/7fa06d8b-464b-4050-a0fd-d319cc509390/18fa9a6d-388b-4829-a409-257b50720dd4"
-					(reference "#PWR0358")
+					(reference "#PWR0360")
 					(unit 1)
 				)
@@
 			(project "vootington V4N"
 				(path "/7fa06d8b-464b-4050-a0fd-d319cc509390/18fa9a6d-388b-4829-a409-257b50720dd4"
-					(reference "#PWR0359")
+					(reference "#PWR0361")
 					(unit 1)
 				)
@@
 		(on_board yes)
 		(dnp no)
-		(property "Reference" "C125"
+		(property "Reference" "C124"
 			(at 162.052 121.666 90)
 			(effects
@@
 			(project "vootington V4N V2"
 				(path "/7fa06d8b-464b-4050-a0fd-d319cc509390/18fa9a6d-388b-4829-a409-257b50720dd4"
-					(reference "C125")
+					(reference "C124")
 					(unit 1)
 				)
@@
 		(dnp no)
 		(fields_autoplaced yes)
-		(property "Reference" "#PWR0371"
+		(property "Reference" "#PWR0373"
 			(at 102.87 124.46 0)
 			(effects
@@
 			(project "vootington V4N V2"
 				(path "/7fa06d8b-464b-4050-a0fd-d319cc509390/18fa9a6d-388b-4829-a409-257b50720dd4"
-					(reference "#PWR0371")
+					(reference "#PWR0373")
 					(unit 1)
 				)
@@
 			(project "vootington V4N"
 				(path "/7fa06d8b-464b-4050-a0fd-d319cc509390/18fa9a6d-388b-4829-a409-257b50720dd4"
-					(reference "#PWR0378")
+					(reference "#PWR0380")
 					(unit 1)
 				)
@@
 			(project "vootington V4N"
 				(path "/7fa06d8b-464b-4050-a0fd-d319cc509390/18fa9a6d-388b-4829-a409-257b50720dd4"
-					(reference "#PWR0374")
+					(reference "#PWR0376")
 					(unit 1)
 				)
@@
 		(dnp no)
 		(fields_autoplaced yes)
-		(property "Reference" "#PWR0372"
+		(property "Reference" "#PWR0374"
 			(at 157.48 124.46 0)
 			(effects
@@
 			(project "vootington V4N V2"
 				(path "/7fa06d8b-464b-4050-a0fd-d319cc509390/18fa9a6d-388b-4829-a409-257b50720dd4"
-					(reference "#PWR0372")
+					(reference "#PWR0374")
 					(unit 1)
 				)
@@
 			(project "vootington V4N"
 				(path "/7fa06d8b-464b-4050-a0fd-d319cc509390/18fa9a6d-388b-4829-a409-257b50720dd4"
-					(reference "#PWR0375")
+					(reference "#PWR0377")
 					(unit 1)
 				)
@@
 			(project "vootington V4N"
 				(path "/7fa06d8b-464b-4050-a0fd-d319cc509390/18fa9a6d-388b-4829-a409-257b50720dd4"
-					(reference "#PWR0380")
+					(reference "#PWR0382")
 					(unit 1)
 				)
@@
 		(dnp no)
 		(fields_autoplaced yes)
-		(property "Reference" "#PWR0352"
+		(property "Reference" "#PWR0354"
 			(at 39.37 22.86 0)
 			(effects
@@
 			(project "vootington V4N V2"
 				(path "/7fa06d8b-464b-4050-a0fd-d319cc509390/18fa9a6d-388b-4829-a409-257b50720dd4"
-					(reference "#PWR0352")
+					(reference "#PWR0354")
 					(unit 1)
 				)
@@
 		(dnp no)
 		(fields_autoplaced yes)
-		(property "Reference" "#PWR0361"
+		(property "Reference" "#PWR0363"
 			(at 102.87 73.66 0)
 			(effects
@@
 			(project "vootington V4N V2"
 				(path "/7fa06d8b-464b-4050-a0fd-d319cc509390/18fa9a6d-388b-4829-a409-257b50720dd4"
-					(reference "#PWR0361")
+					(reference "#PWR0363")
 					(unit 1)
 				)
@@
 			(project "vootington V4N"
 				(path "/7fa06d8b-464b-4050-a0fd-d319cc509390/18fa9a6d-388b-4829-a409-257b50720dd4"
-					(reference "#PWR0351")
+					(reference "#PWR0353")
 					(unit 1)
 				)
@@
 		(dnp no)
 		(fields_autoplaced yes)
-		(property "Reference" "#PWR0370"
+		(property "Reference" "#PWR0372"
 			(at 39.37 124.46 0)
 			(effects
@@
 			(project "vootington V4N V2"
 				(path "/7fa06d8b-464b-4050-a0fd-d319cc509390/18fa9a6d-388b-4829-a409-257b50720dd4"
-					(reference "#PWR0370")
+					(reference "#PWR0372")
 					(unit 1)
 				)
@@
 		(on_board yes)
 		(dnp no)
-		(property "Reference" "C119"
+		(property "Reference" "C118"
 			(at 43.942 20.066 90)
 			(effects
@@
 			(project "vootington V4N V2"
 				(path "/7fa06d8b-464b-4050-a0fd-d319cc509390/18fa9a6d-388b-4829-a409-257b50720dd4"
-					(reference "C119")
+					(reference "C118")
 					(unit 1)
 				)
@@
 			(project "vootington V4N"
 				(path "/7fa06d8b-464b-4050-a0fd-d319cc509390/18fa9a6d-388b-4829-a409-257b50720dd4"
-					(reference "#PWR0357")
+					(reference "#PWR0359")
 					(unit 1)
 				)
@@
 			(project "vootington V4N"
 				(path "/7fa06d8b-464b-4050-a0fd-d319cc509390/18fa9a6d-388b-4829-a409-257b50720dd4"
-					(reference "#PWR0376")
+					(reference "#PWR0378")
 					(unit 1)
 				)
@@
 		(on_board yes)
 		(dnp no)
-		(property "Reference" "C121"
+		(property "Reference" "C120"
 			(at 43.942 70.866 90)
 			(effects
@@
 			(project "vootington V4N V2"
 				(path "/7fa06d8b-464b-4050-a0fd-d319cc509390/18fa9a6d-388b-4829-a409-257b50720dd4"
-					(reference "C121")
+					(reference "C120")
 					(unit 1)
 				)
@@
 			(project "vootington V4N"
 				(path "/7fa06d8b-464b-4050-a0fd-d319cc509390/18fa9a6d-388b-4829-a409-257b50720dd4"
-					(reference "#PWR0354")
+					(reference "#PWR0356")
 					(unit 1)
 				)
@@
 		(on_board yes)
 		(dnp no)
-		(property "Reference" "C124"
+		(property "Reference" "C123"
 			(at 107.442 121.666 90)
 			(effects
@@
 			(project "vootington V4N V2"
 				(path "/7fa06d8b-464b-4050-a0fd-d319cc509390/18fa9a6d-388b-4829-a409-257b50720dd4"
-					(reference "C124")
+					(reference "C123")
 					(unit 1)
 				)
@@
 			(project "vootington V4N"
 				(path "/7fa06d8b-464b-4050-a0fd-d319cc509390/18fa9a6d-388b-4829-a409-257b50720dd4"
-					(reference "#PWR0379")
+					(reference "#PWR0381")
 					(unit 1)
 				)
@@
 			(project "vootington V4N"
 				(path "/7fa06d8b-464b-4050-a0fd-d319cc509390/18fa9a6d-388b-4829-a409-257b50720dd4"
-					(reference "#PWR0367")
+					(reference "#PWR0369")
 					(unit 1)
 				)
@@
 			(project "vootington V4N"
 				(path "/7fa06d8b-464b-4050-a0fd-d319cc509390/18fa9a6d-388b-4829-a409-257b50720dd4"
-					(reference "#PWR0377")
+					(reference "#PWR0379")
 					(unit 1)
 				)
@@
 		(dnp no)
 		(fields_autoplaced yes)
-		(property "Reference" "#PWR0360"
+		(property "Reference" "#PWR0362"
 			(at 39.37 73.66 0)
 			(effects
@@
 			(project "vootington V4N V2"
 				(path "/7fa06d8b-464b-4050-a0fd-d319cc509390/18fa9a6d-388b-4829-a409-257b50720dd4"
-					(reference "#PWR0360")
+					(reference "#PWR0362")
 					(unit 1)
 				)
@@
 			(project "vootington V4N"
 				(path "/7fa06d8b-464b-4050-a0fd-d319cc509390/18fa9a6d-388b-4829-a409-257b50720dd4"
-					(reference "#PWR0364")
+					(reference "#PWR0366")
 					(unit 1)
 				)
@@
 		(dnp no)
 		(fields_autoplaced yes)
-		(property "Reference" "#PWR0353"
+		(property "Reference" "#PWR0355"
 			(at 102.87 22.86 0)
 			(effects
@@
 			(project "vootington V4N V2"
 				(path "/7fa06d8b-464b-4050-a0fd-d319cc509390/18fa9a6d-388b-4829-a409-257b50720dd4"
-					(reference "#PWR0353")
+					(reference "#PWR0355")
 					(unit 1)
 				)
@@
 		(on_board yes)
 		(dnp no)
-		(property "Reference" "C123"
+		(property "Reference" "C122"
 			(at 43.942 121.666 90)
 			(effects
@@
 			(project "vootington V4N V2"
 				(path "/7fa06d8b-464b-4050-a0fd-d319cc509390/18fa9a6d-388b-4829-a409-257b50720dd4"
-					(reference "C123")
+					(reference "C122")
 					(unit 1)
 				)
@@
 		(on_board yes)
 		(dnp no)
-		(property "Reference" "C122"
+		(property "Reference" "C121"
 			(at 107.442 70.866 90)
 			(effects
@@
 			(project "vootington V4N V2"
 				(path "/7fa06d8b-464b-4050-a0fd-d319cc509390/18fa9a6d-388b-4829-a409-257b50720dd4"
-					(reference "C122")
+					(reference "C121")
 					(unit 1)
 				)
@@
 			(project "vootington V4N"
 				(path "/7fa06d8b-464b-4050-a0fd-d319cc509390/18fa9a6d-388b-4829-a409-257b50720dd4"
-					(reference "#PWR0356")
+					(reference "#PWR0358")
 					(unit 1)
 				)
@@
 			(project "vootington V4N"
 				(path "/7fa06d8b-464b-4050-a0fd-d319cc509390/18fa9a6d-388b-4829-a409-257b50720dd4"
-					(reference "#PWR0373")
+					(reference "#PWR0375")
 					(unit 1)
 				)
@@
 		(on_board yes)
 		(dnp no)
-		(property "Reference" "C120"
+		(property "Reference" "C119"
 			(at 107.442 20.066 90)
 			(effects
@@
 			(project "vootington V4N V2"
 				(path "/7fa06d8b-464b-4050-a0fd-d319cc509390/18fa9a6d-388b-4829-a409-257b50720dd4"
-					(reference "C120")
+					(reference "C119")
 					(unit 1)
 				)
@@
 			(project "vootington V4N"
 				(path "/7fa06d8b-464b-4050-a0fd-d319cc509390/18fa9a6d-388b-4829-a409-257b50720dd4"
-					(reference "#PWR0366")
+					(reference "#PWR0368")
 					(unit 1)
 				)
@@
 			(project "vootington V4N"
 				(path "/7fa06d8b-464b-4050-a0fd-d319cc509390/18fa9a6d-388b-4829-a409-257b50720dd4"
-					(reference "#PWR0368")
+					(reference "#PWR0370")
 					(unit 1)
 				)
@@
 			(project "vootington V4N"
 				(path "/7fa06d8b-464b-4050-a0fd-d319cc509390/18fa9a6d-388b-4829-a409-257b50720dd4"
-					(reference "#PWR0362")
+					(reference "#PWR0364")
 					(unit 1)
 				)
@@
 			(project "vootington V4N"
 				(path "/7fa06d8b-464b-4050-a0fd-d319cc509390/18fa9a6d-388b-4829-a409-257b50720dd4"
-					(reference "#PWR0355")
+					(reference "#PWR0357")
 					(unit 1)
 				)
@@
 			(project "vootington V4N"
 				(path "/7fa06d8b-464b-4050-a0fd-d319cc509390/18fa9a6d-388b-4829-a409-257b50720dd4"
-					(reference "#PWR0365")
+					(reference "#PWR0367")
 					(unit 1)
 				)
@@
 			(project "vootington V4N"
 				(path "/7fa06d8b-464b-4050-a0fd-d319cc509390/18fa9a6d-388b-4829-a409-257b50720dd4"
-					(reference "#PWR0369")
+					(reference "#PWR0371")
 					(unit 1)
 				)
@@
 			(project "vootington V4N"
 				(path "/7fa06d8b-464b-4050-a0fd-d319cc509390/18fa9a6d-388b-4829-a409-257b50720dd4"
-					(reference "#PWR0350")
+					(reference "#PWR0352")
 					(unit 1)
 				)
