File: Project/rgb V4N.kicad_sch (KiCad schematic)
At the start: 58 parts, among them U5 74AHCT1G125

Commit message: rgb footprints changed, fresh gerbers, production
Parts:
- D1, D2, D3, D4, D5, D6: footprint PCM_marbastlib-various:LED_6028R -> cipulot_parts:SK6812-MINI-E; symbol PCM_marbastlib-various:SK6812MINI-E -> cipulot_parts:YS-SK6812MINI-E
Connections:
- net GND: now also D1.3 (VSS), D1.3 (VSS), D1.3 (VSS), D1.3 (VSS), D1.3 (VSS), D1.3 (VSS), D1.3 (VSS), D1.3 (VSS), D1.3 (VSS), D1.3 (VSS), D2.3 (VSS), D2.3 (VSS), D2.3 (VSS), D2.3 (VSS), D2.3 (VSS), D2.3 (VSS), D2.3 (VSS), D2.3 (VSS), D2.3 (VSS), D2.3 (VSS), D3.3 (VSS), D3.3 (VSS), D3.3 (VSS), D3.3 (VSS), D3.3 (VSS), D3.3 (VSS), D3.3 (VSS), D3.3 (VSS), D3.3 (VSS), D3.3 (VSS), D4.3 (VSS), D4.3 (VSS), D4.3 (VSS), D4.3 (VSS), D4.3 (VSS), D4.3 (VSS), D4.3 (VSS), D4.3 (VSS), D5.3 (VSS), D5.3 (VSS), D5.3 (VSS), D5.3 (VSS), D5.3 (VSS), D5.3 (VSS), D5.3 (VSS), D5.3 (VSS), D5.3 (VSS), D6.3 (VSS), D6.3 (VSS), D6.3 (VSS), D6.3 (VSS), D6.3 (VSS), D6.3 (VSS), D6.3 (VSS), D6.3 (VSS), D6.3 (VSS); no longer D1.4 (VSS), D1.4 (VSS), D1.4 (VSS), D1.4 (VSS), D1.4 (VSS), D1.4 (VSS), D1.4 (VSS), D1.4 (VSS), D1.4 (VSS), D1.4 (VSS), D2.4 (VSS), D2.4 (VSS), D2.4 (VSS), D2.4 (VSS), D2.4 (VSS), D2.4 (VSS), D2.4 (VSS), D2.4 (VSS), D2.4 (VSS), D2.4 (VSS), D3.4 (VSS), D3.4 (VSS), D3.4 (VSS), D3.4 (VSS), D3.4 (VSS), D3.4 (VSS), D3.4 (VSS), D3.4 (VSS), D3.4 (VSS), D3.4 (VSS), D4.4 (VSS), D4.4 (VSS), D4.4 (VSS), D4.4 (VSS), D4.4 (VSS), D4.4 (VSS), D4.4 (VSS), D4.4 (VSS), D5.4 (VSS), D5.4 (VSS), D5.4 (VSS), D5.4 (VSS), D5.4 (VSS), D5.4 (VSS), D5.4 (VSS), D5.4 (VSS), D5.4 (VSS), D6.4 (VSS), D6.4 (VSS), D6.4 (VSS), D6.4 (VSS), D6.4 (VSS), D6.4 (VSS), D6.4 (VSS), D6.4 (VSS), D6.4 (VSS)
- net RGB: now also D3.4 (DIN); no longer D3.3 (DIN)
- net at D4.2 (DOUT): now also D6.4 (DIN); no longer D6.3 (DIN) (x7)
- net at D1.2 (DOUT): now also D4.4 (DIN); no longer D4.3 (DIN) (x8)
- net at D3.2 (DOUT): now also D2.4 (DIN); no longer D2.3 (DIN) (x10)
- net at D5.2 (DOUT): now also D3.4 (DIN); no longer D3.3 (DIN) (x9)
- net at D6.2 (DOUT): now also D5.4 (DIN); no longer D5.3 (DIN) (x9)
- net at D2.2 (DOUT): now also D1.4 (DIN); no longer D1.3 (DIN) (x9)
- net at D1.2 (DOUT): now also D6.4 (DIN); no longer D6.3 (DIN) (x2)
- net at D4.2 (DOUT): now also D1.4 (DIN); no longer D1.3 (DIN)

Commit message: update
Parts:
- D1, D2, D3, D4, D5, D6: value SK6812MINI-E -> YS-SK6803MINI-E; footprint cipulot_parts:SK6812-MINI-E -> cipulot_parts:SK6803-MINI-E; symbol cipulot_parts:YS-SK6812MINI-E -> cipulot_parts:YS-SK6803MINI-E
Connections:
- net +5V: now also D1.3 (VDD), D1.3 (VDD), D1.3 (VDD), D1.3 (VDD), D1.3 (VDD), D1.3 (VDD), D1.3 (VDD), D1.3 (VDD), D1.3 (VDD), D1.3 (VDD), D2.3 (VDD), D2.3 (VDD), D2.3 (VDD), D2.3 (VDD), D2.3 (VDD), D2.3 (VDD), D2.3 (VDD), D2.3 (VDD), D2.3 (VDD), D2.3 (VDD), D3.3 (VDD), D3.3 (VDD), D3.3 (VDD), D3.3 (VDD), D3.3 (VDD), D3.3 (VDD), D3.3 (VDD), D3.3 (VDD), D3.3 (VDD), D3.3 (VDD), D4.3 (VDD), D4.3 (VDD), D4.3 (VDD), D4.3 (VDD), D4.3 (VDD), D4.3 (VDD), D4.3 (VDD), D4.3 (VDD), D5.3 (VDD), D5.3 (VDD), D5.3 (VDD), D5.3 (VDD), D5.3 (VDD), D5.3 (VDD), D5.3 (VDD), D5.3 (VDD), D5.3 (VDD), D6.3 (VDD), D6.3 (VDD), D6.3 (VDD), D6.3 (VDD), D6.3 (VDD), D6.3 (VDD), D6.3 (VDD), D6.3 (VDD), D6.3 (VDD); no longer D1.1 (VDD), D1.1 (VDD), D1.1 (VDD), D1.1 (VDD), D1.1 (VDD), D1.1 (VDD), D1.1 (VDD), D1.1 (VDD), D1.1 (VDD), D1.1 (VDD), D2.1 (VDD), D2.1 (VDD), D2.1 (VDD), D2.1 (VDD), D2.1 (VDD), D2.1 (VDD), D2.1 (VDD), D2.1 (VDD), D2.1 (VDD), D2.1 (VDD), D3.1 (VDD), D3.1 (VDD), D3.1 (VDD), D3.1 (VDD), D3.1 (VDD), D3.1 (VDD), D3.1 (VDD), D3.1 (VDD), D3.1 (VDD), D3.1 (VDD), D4.1 (VDD), D4.1 (VDD), D4.1 (VDD), D4.1 (VDD), D4.1 (VDD), D4.1 (VDD), D4.1 (VDD), D4.1 (VDD), D5.1 (VDD), D5.1 (VDD), D5.1 (VDD), D5.1 (VDD), D5.1 (VDD), D5.1 (VDD), D5.1 (VDD), D5.1 (VDD), D5.1 (VDD), D6.1 (VDD), D6.1 (VDD), D6.1 (VDD), D6.1 (VDD), D6.1 (VDD), D6.1 (VDD), D6.1 (VDD), D6.1 (VDD), D6.1 (VDD)
- net GND: now also D1.1 (VSS), D1.1 (VSS), D1.1 (VSS), D1.1 (VSS), D1.1 (VSS), D1.1 (VSS), D1.1 (VSS), D1.1 (VSS), D1.1 (VSS), D1.1 (VSS), D2.1 (VSS), D2.1 (VSS), D2.1 (VSS), D2.1 (VSS), D2.1 (VSS), D2.1 (VSS), D2.1 (VSS), D2.1 (VSS), D2.1 (VSS), D2.1 (VSS), D3.1 (VSS), D3.1 (VSS), D3.1 (VSS), D3.1 (VSS), D3.1 (VSS), D3.1 (VSS), D3.1 (VSS), D3.1 (VSS), D3.1 (VSS), D3.1 (VSS), D4.1 (VSS), D4.1 (VSS), D4.1 (VSS), D4.1 (VSS), D4.1 (VSS), D4.1 (VSS), D4.1 (VSS), D4.1 (VSS), D5.1 (VSS), D5.1 (VSS), D5.1 (VSS), D5.1 (VSS), D5.1 (VSS), D5.1 (VSS), D5.1 (VSS), D5.1 (VSS), D5.1 (VSS), D6.1 (VSS), D6.1 (VSS), D6.1 (VSS), D6.1 (VSS), D6.1 (VSS), D6.1 (VSS), D6.1 (VSS), D6.1 (VSS), D6.1 (VSS); no longer D1.3 (VSS), D1.3 (VSS), D1.3 (VSS), D1.3 (VSS), D1.3 (VSS), D1.3 (VSS), D1.3 (VSS), D1.3 (VSS), D1.3 (VSS), D1.3 (VSS), D2.3 (VSS), D2.3 (VSS), D2.3 (VSS), D2.3 (VSS), D2.3 (VSS), D2.3 (VSS), D2.3 (VSS), D2.3 (VSS), D2.3 (VSS), D2.3 (VSS), D3.3 (VSS), D3.3 (VSS), D3.3 (VSS), D3.3 (VSS), D3.3 (VSS), D3.3 (VSS), D3.3 (VSS), D3.3 (VSS), D3.3 (VSS), D3.3 (VSS), D4.3 (VSS), D4.3 (VSS), D4.3 (VSS), D4.3 (VSS), D4.3 (VSS), D4.3 (VSS), D4.3 (VSS), D4.3 (VSS), D5.3 (VSS), D5.3 (VSS), D5.3 (VSS), D5.3 (VSS), D5.3 (VSS), D5.3 (VSS), D5.3 (VSS), D5.3 (VSS), D5.3 (VSS), D6.3 (VSS), D6.3 (VSS), D6.3 (VSS), D6.3 (VSS), D6.3 (VSS), D6.3 (VSS), D6.3 (VSS), D6.3 (VSS), D6.3 (VSS)
- net RGB: now also D3.2 (DIN); no longer D3.4 (DIN)
- net at D4.2 (DIN): now also D1.4 (DOUT); no longer D6.4 (DIN) (x3)
- net at D4.4 (DOUT): now also D6.2 (DIN); no longer D1.2 (DOUT) (x3)
- net at D3.2 (DIN): now also D5.4 (DOUT); no longer D2.4 (DIN) (x3)
- net at D3.4 (DOUT): now also D2.2 (DIN); no longer D5.2 (DOUT) (x3)
- net at D5.2 (DIN): now also D6.4 (DOUT); no longer D3.4 (DIN) (x5)
- net at D5.4 (DOUT): now also D3.2 (DIN); no longer D6.2 (DOUT) (x5)
- net at D1.2 (DIN): now also D2.4 (DOUT); no longer D4.4 (DIN) (x4)
- net at D1.4 (DOUT): now also D4.2 (DIN); no longer D2.2 (DOUT) (x4)
- net at D1.2 (DIN): now also D2.4 (DOUT); no longer D6.4 (DIN)
- net at D1.4 (DOUT): now also D6.2 (DIN); no longer D2.2 (DOUT)
- net at D6.2 (DIN): now also D4.4 (DOUT); no longer D5.4 (DIN) (x3)
- net at D6.4 (DOUT): now also D5.2 (DIN); no longer D4.2 (DOUT) (x3)
- net at D2.2 (DIN): now also D3.4 (DOUT); no longer D1.4 (DIN) (x4)
- net at D2.4 (DOUT): now also D1.2 (DIN); no longer D3.2 (DOUT) (x4)
- net at D1.2 (DIN): now also D4.4 (DOUT); no longer D6.4 (DIN)
- net at D1.4 (DOUT): now also D6.2 (DIN); no longer D4.2 (DOUT)
- new net: D2.2 (DIN), D3.4 (DOUT) (x3)
- new net: D5.2 (DIN), D6.4 (DOUT)
- new net: D3.2 (DIN), D5.4 (DOUT)
- new net: D4.4 (DOUT), D6.2 (DIN)
- new net: D1.4 (DOUT), D4.2 (DIN)

Commit message: revision work
Parts:
- removed D4: YS-SK6803MINI-E, cipulot_parts:SK6803-MINI-E, symbol cipulot_parts:YS-SK6803MINI-E
- added C100, C101, C102, C103, C104, C105, C106, C107, C108, C109, C110, C111, C112, C113, C114, C115, C116, C117, C118, C63, C64, C65, C67, C68, C69, C70, C71, C72, C73, C74, C75, C76, C77, C78, C79, C80, C81, C82, C83, C84, C85, C86, C87, C88, C89, C90, C91, C92, C93, C94, C95, C96, C97, C98, C99: 100nF, Capacitor_SMD:C_0402_1005Metric, symbol Device:C_Small
Connections:
- net +5V: now also C100.1, C101.1, C102.1, C103.1, C104.1, C105.1, C106.1, C107.1, C108.1, C109.1, C110.1, C111.1, C112.1, C113.1, C114.1, C115.1, C116.1, C117.1, C118.1, C63.1, C64.1, C65.1, C67.1, C68.1, C69.1, C70.1, C71.1, C72.1, C73.1, C74.1, C75.1, C76.1, C77.1, C78.1, C79.1, C80.1, C81.1, C82.1, C83.1, C84.1, C85.1, C86.1, C87.1, C88.1, C89.1, C90.1, C91.1, C92.1, C93.1, C94.1, C95.1, C96.1, C97.1, C98.1, C99.1
- net GND: now also C100.2, C101.2, C102.2, C103.2, C104.2, C105.2, C106.2, C107.2, C108.2, C109.2, C110.2, C111.2, C112.2, C113.2, C114.2, C115.2, C116.2, C117.2, C118.2, C63.2, C64.2, C65.2, C67.2, C68.2, C69.2, C70.2, C71.2, C72.2, C73.2, C74.2, C75.2, C76.2, C77.2, C78.2, C79.2, C80.2, C81.2, C82.2, C83.2, C84.2, C85.2, C86.2, C87.2, C88.2, C89.2, C90.2, C91.2, C92.2, C93.2, C94.2, C95.2, C96.2, C97.2, C98.2, C99.2
- net at D1.2 (DIN): now also D1.4 (DOUT)

Commit message: backups
Parts:
- renumbered C101 to C100, C102 to C101, C103 to C102, C104 to C103, C105 to C104, C106 to C105, C107 to C106, C108 to C107, C109 to C108, C110 to C109, C111 to C110, C112 to C111, C113 to C112, C114 to C113, C115 to C114, C116 to C115, C117 to C116, C118 to C117, C63 to C62, C64 to C63, C65 to C64, C67 to C66, C68 to C67, C69 to C68, C70 to C69, C71 to C70, C72 to C71, C73 to C72, C74 to C73, C75 to C74, C76 to C75, C77 to C76, C78 to C77, C79 to C78, C80 to C79, C81 to C80, C82 to C81, C83 to C82, C84 to C83, C85 to C84, C86 to C85, C87 to C86, C88 to C87, C89 to C88, C90 to C89, C91 to C90, C92 to C91, C93 to C92, C94 to C93, C95 to C94, C96 to C95, C97 to C96, C98 to C97, C99 to C98, C100 to C99
