File: Project/MCU V4N STM32G0B1CBT6.kicad_sch (KiCad schematic)
At the start: 14 parts, among them J1 Conn_01x04, U65 STM32G0B1CBTx

Commit message: backups
Parts:
- renumbered C126 to C53, C127 to C54, C128 to C55, R4 to R1, R5 to R2, R7 to R3, R6 to R4, U65 to U53
Changed lines of the file:
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@@
 			(project "vootington V4N STM32G0B1CBT6"
 				(path "/7fa06d8b-464b-4050-a0fd-d319cc509390/00617548-7095-421c-9d05-30ad704b65f1"
-					(reference "#PWR0163")
+					(reference "#PWR0165")
 					(unit 1)
 				)
@@
 		(on_board yes)
 		(dnp no)
-		(property "Reference" "C126"
+		(property "Reference" "C53"
 			(at 89.281 44.5516 0)
 			(effects
@@
 			(project "vootington V4N STM32G0B1CBT6"
 				(path "/7fa06d8b-464b-4050-a0fd-d319cc509390/00617548-7095-421c-9d05-30ad704b65f1"
-					(reference "C126")
+					(reference "C53")
 					(unit 1)
 				)
@@
 			(project "vootington V4N STM32G0B1CBT6"
 				(path "/7fa06d8b-464b-4050-a0fd-d319cc509390/00617548-7095-421c-9d05-30ad704b65f1"
-					(reference "R1")
+					(reference "R5")
 					(unit 1)
 				)
@@
 		(on_board yes)
 		(dnp no)
-		(property "Reference" "R5"
+		(property "Reference" "R2"
 			(at 160.02 52.07 90)
 			(effects
@@
 			(project "vootington V4N STM32G0B1CBT6"
 				(path "/7fa06d8b-464b-4050-a0fd-d319cc509390/00617548-7095-421c-9d05-30ad704b65f1"
-					(reference "R5")
+					(reference "R2")
 					(unit 1)
 				)
@@
 		(dnp no)
 		(fields_autoplaced yes)
-		(property "Reference" "U65"
+		(property "Reference" "U53"
 			(at 46.6441 121.92 0)
 			(effects
@@
 			(project "vootington V4N STM32G0B1CBT6"
 				(path "/7fa06d8b-464b-4050-a0fd-d319cc509390/00617548-7095-421c-9d05-30ad704b65f1"
-					(reference "U65")
+					(reference "U53")
 					(unit 1)
 				)
@@
 		(dnp no)
 		(fields_autoplaced yes)
-		(property "Reference" "R7"
+		(property "Reference" "R3"
 			(at 163.83 68.5799 0)
 			(effects
@@
 			(project "vootington V4N STM32G0B1CBT6"
 				(path "/7fa06d8b-464b-4050-a0fd-d319cc509390/00617548-7095-421c-9d05-30ad704b65f1"
-					(reference "R7")
+					(reference "R3")
 					(unit 1)
 				)
@@
 		(on_board yes)
 		(dnp no)
-		(property "Reference" "R6"
+		(property "Reference" "R4"
 			(at 90.17 78.74 90)
 			(effects
@@
 			(project "vootington V4N STM32G0B1CBT6"
 				(path "/7fa06d8b-464b-4050-a0fd-d319cc509390/00617548-7095-421c-9d05-30ad704b65f1"
-					(reference "R6")
+					(reference "R4")
 					(unit 1)
 				)
@@
 		(on_board yes)
 		(dnp no)
-		(property "Reference" "C127"
+		(property "Reference" "C54"
 			(at 104.521 44.5516 0)
 			(effects
@@
 			(project "vootington V4N STM32G0B1CBT6"
 				(path "/7fa06d8b-464b-4050-a0fd-d319cc509390/00617548-7095-421c-9d05-30ad704b65f1"
-					(reference "C127")
+					(reference "C54")
 					(unit 1)
 				)
@@
 		(dnp no)
 		(fields_autoplaced yes)
-		(property "Reference" "#PWR0382"
+		(property "Reference" "#PWR0157"
 			(at 43.18 30.48 0)
 			(effects
@@
 			(project "vootington V4N STM32G0B1CBT6"
 				(path "/7fa06d8b-464b-4050-a0fd-d319cc509390/00617548-7095-421c-9d05-30ad704b65f1"
-					(reference "#PWR0382")
+					(reference "#PWR0157")
 					(unit 1)
 				)
@@
 		(on_board yes)
 		(dnp no)
-		(property "Reference" "C128"
+		(property "Reference" "C55"
 			(at 117.221 44.5516 0)
 			(effects
@@
 			(project "vootington V4N STM32G0B1CBT6"
 				(path "/7fa06d8b-464b-4050-a0fd-d319cc509390/00617548-7095-421c-9d05-30ad704b65f1"
-					(reference "C128")
+					(reference "C55")
 					(unit 1)
 				)
@@
 		(dnp no)
 		(fields_autoplaced yes)
-		(property "Reference" "R4"
+		(property "Reference" "R1"
 			(at 160.02 39.37 90)
 			(effects
@@
 			(project "vootington V4N STM32G0B1CBT6"
 				(path "/7fa06d8b-464b-4050-a0fd-d319cc509390/00617548-7095-421c-9d05-30ad704b65f1"
-					(reference "R4")
+					(reference "R1")
 					(unit 1)
 				)
@@
 		(dnp no)
 		(fields_autoplaced yes)
-		(property "Reference" "#PWR0383"
+		(property "Reference" "#PWR0161"
 			(at 86.36 58.42 0)
 			(effects
@@
 			(project "vootington V4N STM32G0B1CBT6"
 				(path "/7fa06d8b-464b-4050-a0fd-d319cc509390/00617548-7095-421c-9d05-30ad704b65f1"
-					(reference "#PWR0383")
+					(reference "#PWR0161")
 					(unit 1)
 				)
@@
 			(project "vootington V4N STM32G0B1CBT6"
 				(path "/7fa06d8b-464b-4050-a0fd-d319cc509390/00617548-7095-421c-9d05-30ad704b65f1"
-					(reference "#PWR0162")
+					(reference "#PWR0160")
 					(unit 1)
 				)
@@
 		(on_board yes)
 		(dnp no)
-		(property "Reference" "#PWR0160"
+		(property "Reference" "#PWR0163"
 			(at 86.36 74.93 0)
 			(effects
@@
 			(project "vootington V4N STM32G0B1CBT6"
 				(path "/7fa06d8b-464b-4050-a0fd-d319cc509390/00617548-7095-421c-9d05-30ad704b65f1"
-					(reference "#PWR0160")
+					(reference "#PWR0163")
 					(unit 1)
 				)
@@
 		(dnp no)
 		(fields_autoplaced yes)
-		(property "Reference" "#PWR0159"
+		(property "Reference" "#PWR0162"
 			(at 161.29 68.58 0)
 			(effects
@@
 			(project "vootington V4N STM32G0B1CBT6"
 				(path "/7fa06d8b-464b-4050-a0fd-d319cc509390/00617548-7095-421c-9d05-30ad704b65f1"
-					(reference "#PWR0159")
+					(reference "#PWR0162")
 					(unit 1)
 				)
@@
 		(dnp no)
 		(fields_autoplaced yes)
-		(property "Reference" "#PWR0161"
+		(property "Reference" "#PWR0159"
 			(at 165.1 45.72 0)
 			(effects
@@
 			(project "vootington V4N STM32G0B1CBT6"
 				(path "/7fa06d8b-464b-4050-a0fd-d319cc509390/00617548-7095-421c-9d05-30ad704b65f1"
-					(reference "#PWR0161")
+					(reference "#PWR0159")
 					(unit 1)
 				)
@@
 		(dnp no)
 		(fields_autoplaced yes)
-		(property "Reference" "#PWR0381"
+		(property "Reference" "#PWR0166"
 			(at 44.45 128.27 0)
 			(effects
@@
 			(project "vootington V4N STM32G0B1CBT6"
 				(path "/7fa06d8b-464b-4050-a0fd-d319cc509390/00617548-7095-421c-9d05-30ad704b65f1"
-					(reference "#PWR0381")
+					(reference "#PWR0166")
 					(unit 1)
 				)
@@
 			(project "vootington V4N STM32G0B1CBT6"
 				(path "/7fa06d8b-464b-4050-a0fd-d319cc509390/00617548-7095-421c-9d05-30ad704b65f1"
-					(reference "C59")
-					(unit 1)
-				)
+					(reference "C56")
+					(unit 1)
+				)
